File: hardware/eagle/bbb-cc2520/rev_a/bbb-cc2520_a.brd (EAGLE design)
At the start: 54.6 x 86.4 mm, 32 parts, among them P1 MOLEX_73251-135X, P9/P8 BBB_HEADERS, U1 CC2520, U2 CAT24C256WI-GT3, X1 NX2520SA

Commit message: finished routing both radios, rf traces
Parts:
- added C10, C11, C13, C9: 100nF, rcl:C0402
- added C12: 1uF, rcl:C0603
- added C14, C15: 27pF, rcl:C0402
- added C16: 3pF, rcl:C0402
- added C17: 3.9pF, rcl:C0402
- added C18, C19, C21: 1nF, rcl:C0402
- added C20: 15pF, rcl:C0402
- added C23: 2.2uF, rcl:C0402
- added C24: 2.7pF, rcl:C0402
- added C25: 1pF, rcl:C0402
- added C26: 6.8pF, rcl:C0402
- added IC1: CC2591, bbb-cc2520:PVQFN-16
- added L10: 1kOhm, SparkFun-Passives:C0402
- added L11: 1.5nH, SparkFun-Passives:C0402
- added L12, L3, L5, L6: 1nH, SparkFun-Passives:C0402
- added L2: (no value), SparkFun-Passives:0603
- added L4: 2nH, SparkFun-Passives:C0402
- added L7: (no value), SparkFun-Passives:C0402
- added L8: 1.1nH, SparkFun-Passives:C0402
- added L9: 5.1nH, SparkFun-Passives:C0402
- added P2: MOLEX_73251-135X, connector:SMA-J/PCB
- added R12: 1M 1%, rcl:R0402
- added R13: 56k 1%, rcl:R0402
- added R14: 4.3k, rcl:R0402
- added R15, R16: 1k 1%, rcl:R0402
- added R17: 330k 1%, rcl:R0402
- added U5: CC2520, chips:S-PVQFN-N28
- added X2: NX2520SA, rpi-cc2520:NX2520SA
- C4: value 100nF -> 1uF; device rcl:C0402 -> rcl:C0603
- C5: value 1uF -> 100nF; device rcl:C0603 -> rcl:C0402
- moved C4 13.2 mm to (11.2, 10.9), turned to 180 degrees
- moved C5 12.0 mm to (21.6, 19.1), turned to 0 degrees
- moved C3 11.7 mm to (13.3, 20.3), turned to 0 degrees
- moved C2 10.6 mm to (21.6, 13.7), turned to 270 degrees
- moved C1 7.55 mm to (11.2, 13.1), turned to 180 degrees
- moved R4 4.84 mm to (18.9, 21.3), turned to 180 degrees
- moved R6 3.81 mm to (11.4, 76.8)
- moved R8 3.81 mm to (11.4, 73.0)
- moved U$1 1.08 mm to (46.5, 3.94)
- moved P1 0.25 mm to (18.0, 4.65)
Connections:
- net !RESET renamed !RESET0
- net CCA renamed CCA0
- net CC_GPIO0 renamed CC_GPIO0_0
- net CC_GPIO5 renamed CC_GPIO5_0
- net CE0 renamed CS0
- removed net FIFO: P9/P8.P8_11, U1.9
- removed net FIFOP: P9/P8.P8_12, U1.7
- removed net SFD: P9/P8.P8_15, U1.5
- new net !RESET1: P9/P8.P8_26, U5.25
- new net CCA1: P9/P8.P8_12, U5.6
- new net CS1: P9/P8.P9_16, U5.3
- new net EN: R16.2, U5.10
- new net FIFO0: P9/P8.P9_27, U1.9
- new net FIFO1: P9/P8.P8_14, U5.9
- new net FIFOP0: P9/P8.P9_23, U1.7
- new net FIFOP1: P9/P8.P8_11, U5.7
- new net N$44: IC1.4, L4.1, L7.1
- new net N$45: IC1.2, L3.1, L7.2
- new net N$46: C17.2, L3.2, L6.2
- new net N$47: C16.2, L4.2, L5.2
- new net N$48: IC1.10, L8.1, L9.1
- new net N$49: C18.1, C19.1, C21.1, C23.1, IC1.1, IC1.13, IC1.16, L10.2, L9.2
- new net N$50: C20.1, L8.2
- new net N$51: IC1.11, L11.2
- new net N$52: C24.1, C26.1, L12.1, P2.1
- new net N$53: C25.1, C26.2, L11.1
- new net N$54: IC1.15, R14.2
- new net N$55: IC1.5, R15.1
- new net N$56: IC1.6, R16.1
- new net N$57: C10.1, C11.1, C12.1, C9.1, L2.1, U5.11, U5.14, U5.16, U5.20, U5.22, U5.24, U5.26, U5.8
- new net N$58: C13.1, U5.27
- new net N$59: C15.1, U5.13, X2.1
- new net N$60: C14.1, U5.12, X2.3
- new net N$61: R13.2, U5.23
- new net N$62: IC1.7, R17.1
- new net PAEN: R15.2, U5.4
- new net RF_N2: C17.1, U5.19
- new net RF_P2: C16.1, U5.17
- new net SFD0: P9/P8.P9_14, U1.5
- new net SFD1: P9/P8.P8_15, U5.5
- net GND: now also C10.2, C11.2, C12.2, C13.2, C14.2, C15.2, C18.2, C19.2, C20.2, C21.2, C23.2, C24.2, C25.2, C9.2, IC1.12, IC1.14, IC1.8, IC1.9, IC1.PAD, L12.2, L5.1, L6.1, P2.2, P2.3, P2.4, P2.5, R12.1, R13.1, R14.1, U5.THERMALPAD
- net MISO: now also R12.2, U5.1
- net MOSI: now also U5.2
- net N$12: now also C5.1; no longer C4.1
- net N$29: now also R6.1; no longer R8.1
- net N$32: now also R8.1; no longer R6.1
- net N$5: now also C4.1; no longer C5.1
- net SCLK: now also U5.28
- net VCC: now also L10.1, L2.2, R17.2
Routing:
- net FIFO: track 55.2 -> 0.00 mm, vias 2 -> 0
- net FIFOP: track 52.0 -> 0.00 mm, vias 2 -> 0
- net N$57: track 0.00 -> 47.3 mm, vias 0 -> 4
- net SFD: track 46.5 -> 0.00 mm, vias 2 -> 0
- net SCLK: track 28.6 -> 74.2 mm, vias 0 -> 2
- net CS1: track 0.00 -> 44.0 mm, vias 0 -> 2
- net MOSI: track 28.9 -> 69.7 mm, vias 0 -> 2
- net MISO: track 37.1 -> 74.4 mm
- net SFD0: track 0.00 -> 36.7 mm, vias 0 -> 1
- net N$49: track 0.00 -> 35.7 mm, vias 0 -> 5
- net FIFO1: track 0.00 -> 28.2 mm, vias 0 -> 2
- net EN: track 0.00 -> 28.1 mm
- net PAEN: track 0.00 -> 26.5 mm, vias 0 -> 2
- net FIFOP0: track 0.00 -> 25.2 mm
- net GND: track 10.8 -> 34.1 mm, vias 2 -> 18
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
Commit message: finished initial rev a board layout, changes may come soon
Parts:
- R10, R11, R6, R7, R8, R9: device SparkFun-Passives:0402-RES -> rcl:R0402
- moved C7 2.98 mm to (8.13, 14.2), turned to 180 degrees
- moved C15 2.75 mm to (31.2, 31.2), turned to 180 degrees
- moved C6 2.69 mm to (8.13, 19.1), turned to 180 degrees
- moved C14 2.29 mm to (31.2, 35.8), turned to 180 degrees
- moved SJ1 2.03 mm to (17.9, 76.8)
- moved C12 1.93 mm to (33.8, 29.0)
- moved R8 1.89 mm to (13.2, 72.4)
- moved X2 1.83 mm to (32.7, 33.5)
- moved R7 1.80 mm to (13.2, 74.7)
- moved R6 1.78 mm to (13.2, 77.0)
- moved R2 1.55 mm to (47.4, 73.4)
- moved R1 1.55 mm to (42.3, 73.4)
- moved R3 1.55 mm to (52.5, 73.4)
- moved C3 1.48 mm to (12.1, 21.1), turned to 180 degrees
- moved X1 1.30 mm to (9.65, 16.6)
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Routing:
- net GND: track 34.1 -> 21.1 mm, vias 18 -> 239
- net VCC: track 35.5 -> 30.9 mm, vias 8 -> 9
- net LED1: track 32.3 -> 29.9 mm
- net EN: track 28.1 -> 26.2 mm
- net N$32: track 16.6 -> 18.5 mm, vias 0 -> 2
- net N$30: track 12.8 -> 14.5 mm
- net LED2: track 27.9 -> 26.3 mm
- net LED0: track 32.6 -> 31.0 mm
- net FIFO0: track 21.6 -> 23.2 mm, vias 1 -> 0
- net N$49: track 35.7 -> 37.2 mm, vias 5 -> 4
- net N$3: track 1.36 -> 2.81 mm
- net N$2: track 1.36 -> 2.81 mm
- net N$1: track 1.36 -> 2.81 mm
- net N$5: track 53.7 -> 52.3 mm, vias 3 -> 4
- net CS1: track 44.0 -> 42.8 mm
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Other:
- board text added: "!RESET1"
- board text added: "!RST0"
- board text added: "3V3"
- board text added: "5V"
- board text added: "CCA0"
- board text added: "CCA1"
- board text added: "CS0"
- board text added: "CS1"
- board text added: "FIFO0"
- board text added: "FIFO1"
- board text added: "FIFP0"
- board text added: "FIFP1"
- board text added: "GND"
- board text added: "LD0"
- board text added: "LD1"
- board text added: "LD2"
- board text added: "SFD0"
- board text added: "SFD1"
- board text added: "SO"
- board text added: "SPICL"
- board text added: "SYS_5V"

Commit message: fixed labeling and vias
Parts:
- removed C26: 6.8pF, rcl:C0402
- removed L12: 1nH, SparkFun-Passives:C0402
- removed U5: CC2520, chips:S-PVQFN-N28
- added C22: 100nF, rcl:C0402
- added U3: CAT24C256WI-GT3, bbb-cc2520:CAT24C256WI-GT3
- C1: value 100nF -> 1pF
- C10, C8, C9: value 100nF -> 27pF
- C11, C13: value 100nF -> 1nF
- C12: value 1uF -> 1nF; device rcl:C0603 -> rcl:C0402
- C14, C15: value 27pF -> 100nF
- C16: value 3pF -> 100nF
- C17: value 3.9pF -> 100nF
- C18, C19, C21: value 1nF -> 100nF
- C2: value 100nF -> 2.7pF
- C20: value 15pF -> 100nF
- C23: value 2.2uF -> 1uF; device rcl:C0402 -> rcl:C0603
- C24: value 2.7pF -> 1uF; device rcl:C0402 -> rcl:C0603
- C25: value 1pF -> 2.2uF
- C3: value 100nF -> 3pF
- C4: value 1uF -> 6.8pF; device rcl:C0603 -> rcl:C0402
- C5: value 100nF -> 15pF
- C6: value 27pF -> 3.9pF
- L10: value 1kOhm -> 5.1nH
- L11: value 1.5nH -> 1kOhm
- L4: value 2nH -> 1nH
- L7: value (none) -> 1.1nH
- L8: value 1.1nH -> 1.5nH
- L9: value 5.1nH -> 2nH
- R11: value 10k 1% -> 5.6k 5%
- R12: value 1M 1% -> 10k 1%
- R14: value 4.3k -> 56k 1%
- R15: value 1k 1% -> 330k 1%
- R16: value 1k 1% -> 1M 1%
- R17: value 330k 1% -> 1M 1%
- R4: value 1M 1% -> 1k 1%
- R5: value 56k 1% -> 1k 1%
- R6: value 4.75k -> 4.3k
- R9: value 5.6k 5% -> 4.75k
- U2: value CAT24C256WI-GT3 -> CC2520; device bbb-cc2520:CAT24C256WI-GT3 -> chips:S-PVQFN-N28
- moved R6 64.0 mm to (45.5, 21.7)
- moved C8 62.7 mm to (8.13, 14.2)
- moved C18 61.2 mm to (9.14, 77.0), turned to 180 degrees
- moved U2 53.4 mm to (39.4, 35.0), turned to 270 degrees
- moved R12 51.9 mm to (7.62, 80.0), turned to 90 degrees
- moved C6 33.7 mm to (40.1, 29.5), turned to 270 degrees
- moved C14 29.5 mm to (12.2, 13.3)
- moved R13 29.0 mm to (21.6, 15.6)
- moved C1 28.5 mm to (40.6, 15.9), turned to 0 degrees
- moved C4 28.1 mm to (40.0, 14.1), turned to 90 degrees
- moved C16 27.9 mm to (12.1, 21.1), turned to 180 degrees
- moved C3 27.9 mm to (38.7, 29.5), turned to 270 degrees
- moved R17 26.4 mm to (43.7, 43.2)
- moved C23 25.7 mm to (11.9, 11.4)
- moved C17 21.3 mm to (21.6, 19.1), turned to 0 degrees
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Connections:
- net !RESET1: now also U2.25; no longer U5.25
- net CCA1: now also U2.6; no longer U5.6
- net CS1: now also U2.3; no longer U5.3
- net EN: now also R5.2, U2.10; no longer R16.2, U5.10
- net FIFO1: now also U2.9; no longer U5.9
- net FIFOP1: now also U2.7; no longer U5.7
- net GND: now also C16.2, C17.2, C22.2, L3.1, L4.1, L6.2, R16.1, R17.1, R6.1, U2.THERMALPAD, U3.VSS; no longer C3.2, C4.2, C6.2, L12.2, L5.1, L6.1, R12.1, R4.1, R5.1, U2.VSS, U5.THERMALPAD
- net MISO: now also R16.2, R17.2, U2.1; no longer R12.2, R4.2, U5.1
- net MOSI: now also U2.2; no longer U5.2
- net N$11: now also C8.1; no longer C7.1
- net N$12: now also C17.1; no longer C5.1
- net N$13: now also C7.1; no longer C6.1
- net N$14: now also R13.2; no longer R5.2
- net N$29: now also R7.1, U3.A0; no longer R6.1, U2.A0
- net N$30: now also R8.1, U3.A1; no longer R7.1, U2.A1
- net N$31: now also R12.2, U3.WP; no longer R11.2, U2.WP
- net N$32: now also R9.1, U3.A2; no longer R8.1, U2.A2
- net N$44: now also L9.1; no longer L4.1, L7.1
- net N$45: now also L5.1; no longer L3.1, L7.2
- net N$46: now also C6.2, L4.2, L5.2; no longer C17.2, L3.2, L6.2
- net N$47: now also C3.2, L3.2, L9.2; no longer C16.2, L4.2, L5.2
- net N$48: now also L10.1, L7.1; no longer L8.1, L9.1
- net N$49: now also C11.1, C12.1, C13.1, C25.1, L11.2; no longer C18.1, C19.1, C21.1, C23.1, L9.2
- net N$5: now also C14.1, C15.1, C16.1, C23.1; no longer C1.1, C2.1, C3.1, C4.1
- net N$50: now also C5.1, L7.2; no longer C20.1, L8.2
- net N$51: now also L8.2; no longer L11.2
- net N$52: now also C2.1, C4.1, L6.1; no longer C24.1, C26.1, L12.1
- net N$53: now also C1.1, C4.2, L8.1; no longer C25.1, C26.2, L11.1
- net N$54: now also R6.2; no longer R14.2
- net N$55: now also R4.1; no longer R15.1
- net N$56: now also R5.1; no longer R16.1
- net N$57: now also C19.1, C20.1, C21.1, C24.1, U2.11, U2.14, U2.16, U2.20, U2.22, U2.24, U2.26, U2.8; no longer C10.1, C11.1, C12.1, C9.1, U5.11, U5.14, U5.16, U5.20, U5.22, U5.24, U5.26, U5.8
- net N$58: now also C22.1, U2.27; no longer C13.1, U5.27
- net N$59: now also C10.1, U2.13; no longer C15.1, U5.13
- net N$60: now also C9.1, U2.12; no longer C14.1, U5.12
- net N$61: now also R14.2, U2.23; no longer R13.2, U5.23
- net N$62: now also R15.1; no longer R17.1
- net PAEN: now also R4.2, U2.4; no longer R15.2, U5.4
- net RF_N2: now also C6.1, U2.19; no longer C17.1, U5.19
- net RF_P2: now also C3.1, U2.17; no longer C16.1, U5.17
- net SCL: now also R10.1, U3.SCL; no longer R9.1, U2.SCL
- net SCLK: now also U2.28; no longer U5.28
- net SDA: now also R11.1, U3.SDA; no longer R10.1, U2.SDA
- net SFD1: now also U2.5; no longer U5.5
- net VCC: now also C18.1, L11.1, R11.2, R12.1, R15.2, U3.VCC; no longer C8.1, L10.1, R11.1, R17.2, R6.2, U2.VCC
Routing:
- net GND: track 21.1 -> 6.99 mm, vias 239 -> 252
- net MISO: track 73.5 -> 74.6 mm
- net VCC: track 30.9 -> 30.4 mm

Commit message: rev a finished, gerbers generated, bom done
Parts:
- removed U$1: UMICH_SOLID_SMALL, logos:UMICH_SOLID_75MIL
- added U$2: (no value), logos:UMICH_SOLID_200MIL
- renumbered IC1 to U4
Routing:
- net GND: track 6.99 -> 5.76 mm, vias 252 -> 259
