File: hardware/eagle/bbb-cc2520/rev_a/bbb-cc2520_a.sch (EAGLE design)
At the start: 32 parts, among them P1 MOLEX_73251-135X, P9/P8 BBB_HEADERS, U1 CC2520, U2 CAT24C256WI-GT3, X1 NX2520SA

Commit message: finished routing both radios, rf traces
Parts:
- added C10, C11, C13, C9: 100nF, rcl:C-EUC0402
- added C12: 1uF, rcl:C-EUC0603
- added C14, C15: 27pF, rcl:C-EUC0402
- added C16: 3pF, rcl:C-EUC0402
- added C17: 3.9pF, rcl:C-EUC0402
- added C18, C19, C21: 1nF, rcl:C-EUC0402
- added C20: 15pF, rcl:C-EUC0402
- added C23: 2.2uF, rcl:C-EUC0402
- added C24: 2.7pF, rcl:C-EUC0402
- added C25: 1pF, rcl:C-EUC0402
- added C26: 6.8pF, rcl:C-EUC0402
- added IC1: CC2591, bbb-cc2520:CC2591
- added L10: 1kOhm, SparkFun-Passives:INDUCTOR0402
- added L11: 1.5nH, SparkFun-Passives:INDUCTOR0402
- added L12, L3, L5, L6: 1nH, SparkFun-Passives:INDUCTOR0402
- added L2: (no value), SparkFun-Passives:INDUCTOR0603
- added L4: 2nH, SparkFun-Passives:INDUCTOR0402
- added L7: (no value), SparkFun-Passives:INDUCTOR0402
- added L8: 1.1nH, SparkFun-Passives:INDUCTOR0402
- added L9: 5.1nH, SparkFun-Passives:INDUCTOR0402
- added P2: MOLEX_73251-135X, connector:MOLEX_73251-135X
- added R12: 1M 1%, rcl:R-US_R0402
- added R13: 56k 1%, rcl:R-US_R0402
- added R14: 4.3k, rcl:R-US_R0402
- added R15, R16: 1k 1%, rcl:R-US_R0402
- added R17: 330k 1%, rcl:R-US_R0402
- added U5: CC2520, chips:CC2520
- added X2: NX2520SA, rpi-cc2520:NX2520SA
- C4: value 100nF -> 1uF; device rcl:C-EUC0402 -> rcl:C-EUC0603; DIGIKEY 490-1318-1-ND -> 490-1550-1-ND
- C5: value 1uF -> 100nF; device rcl:C-EUC0603 -> rcl:C-EUC0402; DIGIKEY 490-1550-1-ND -> 490-1318-1-ND
Connections:
- net !RESET renamed !RESET0
- net CCA renamed CCA0
- net CC_GPIO0 renamed CC_GPIO0_0
- net CC_GPIO5 renamed CC_GPIO5_0
- net CE0 renamed CS0
- removed net FIFO: P9/P8.GPIO1_13, U1.GPIO1
- removed net FIFOP: P9/P8.GPIO1_12, U1.GPIO2
- removed net SFD: P9/P8.GPIO1_15, U1.GPIO4
- new net !RESET1: P9/P8.GPIO1_29, U5.!RESET
- new net CCA1: P9/P8.GPIO1_12, U5.GPIO3
- new net CS1: P9/P8.EHRPWM1B, U5.!CS
- new net EN: R16.2, U5.GPIO0
- new net FIFO0: P9/P8.GPIO3_19, U1.GPIO1
- new net FIFO1: P9/P8.GPIO0_26, U5.GPIO1
- new net FIFOP0: P9/P8.GPIO1_17, U1.GPIO2
- new net FIFOP1: P9/P8.GPIO1_13, U5.GPIO2
- new net N$44: IC1.RF_P, L4.1, L7.1
- new net N$45: IC1.RF_N, L3.1, L7.2
- new net N$46: C17.2, L3.2, L6.2
- new net N$47: C16.2, L4.2, L5.2
- new net N$48: IC1.AVDD_PA2, L8.1, L9.1
- new net N$49: C18.1, C19.1, C21.1, C23.1, IC1.AVDD_BIAS, IC1.AVDD_LNA, IC1.AVDD_PA1, L10.2, L9.2
- new net N$50: C20.1, L8.2
- new net N$51: IC1.ANT, L11.2
- new net N$52: C24.1, C26.1, L12.1, P2.P$1
- new net N$53: C25.1, C26.2, L11.1
- new net N$54: IC1.BIAS, R14.2
- new net N$55: IC1.PAEN, R15.1
- new net N$56: IC1.EN, R16.1
- new net N$57: C10.1, C11.1, C12.1, C9.1, L2.1, U5.AVDD0, U5.AVDD1, U5.AVDD2, U5.AVDD3, U5.AVDD4, U5.AVDD5, U5.DVDD, U5.VREG_EN
- new net N$58: C13.1, U5.DCOUPL
- new net N$59: C15.1, U5.XOSC_Q1, X2.1
- new net N$60: C14.1, U5.XOSC_Q2, X2.2
- new net N$61: R13.2, U5.RBIAS
- new net N$62: IC1.HGM, R17.1
- new net PAEN: R15.2, U5.GPIO5
- new net RF_N2: C17.1, U5.RF_N
- new net RF_P2: C16.1, U5.RF_P
- new net SFD0: P9/P8.EHRPWM1A, U1.GPIO4
- new net SFD1: P9/P8.GPIO1_15, U5.GPIO4
- net GND: now also C10.2, C11.2, C12.2, C13.2, C14.2, C15.2, C18.2, C19.2, C20.2, C21.2, C23.2, C24.2, C25.2, C9.2, IC1.GND@1, IC1.GND@2, IC1.GND@3, IC1.GND@4, IC1.GND@5, L12.2, L5.1, L6.1, P2.P$2, P2.P$3, P2.P$4, P2.P$5, R12.1, R13.1, R14.1, U5.GND_EXP
- net MISO: now also R12.2, U5.MISO
- net MOSI: now also U5.MOSI
- net N$12: now also C5.1; no longer C4.1
- net N$29: now also R6.1; no longer R8.1
- net N$32: now also R8.1; no longer R6.1
- net N$5: now also C4.1; no longer C5.1
- net SCLK: now also U5.SCLK
- net VCC: now also L10.1, L2.2, R17.2
Other:
- moved on the sheet: C1, C2, C3, C4, C5, R6, R8

Commit message: finished initial rev a board layout, changes may come soon
Parts:
- R10, R11, R6, R7, R8, R9: device SparkFun-Passives:RESISTOR0402-RES -> rcl:R-US_R0402; DIGIKEY (none) -> RHM1.00MCDCT-ND
Changed lines of the file:
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@@
 <part name="SUPPLY2" library="SparkFun-Aesthetics" deviceset="VCC" device=""/>
 <part name="SJ1" library="SparkFun-Passives" deviceset="JUMPER-PAD-3-NO" device="FULL_BOX_SILK"/>
-<part name="R8" library="SparkFun-Passives" deviceset="RESISTOR" device="0402-RES" value="4.75k"/>
-<part name="R7" library="SparkFun-Passives" deviceset="RESISTOR" device="0402-RES" value="4.75k"/>
-<part name="R6" library="SparkFun-Passives" deviceset="RESISTOR" device="0402-RES" value="4.75k"/>
-<part name="R9" library="SparkFun-Passives" deviceset="RESISTOR" device="0402-RES" value="5.6k 5%"/>
-<part name="R10" library="SparkFun-Passives" deviceset="RESISTOR" device="0402-RES" value="5.6k 5%"/>
-<part name="R11" library="SparkFun-Passives" deviceset="RESISTOR" device="0402-RES" value="10k 1%"/>
 <part name="WRT" library="SparkFun-Passives" deviceset="JUMPER-PTH-2-NO" device=""/>
 <part name="GND9" library="SparkFun-Aesthetics" deviceset="GND" device=""/>
@@
 </part>
 <part name="P+6" library="SparkFun" deviceset="VCC" device=""/>
+<part name="R6" library="rcl" deviceset="R-US_" device="R0402" value="4.75k">
+<attribute name="DIGIKEY" value="RHM1.00MCDCT-ND"/>
+</part>
+<part name="R7" library="rcl" deviceset="R-US_" device="R0402" value="4.75k">
+<attribute name="DIGIKEY" value="RHM1.00MCDCT-ND"/>
+</part>
+<part name="R8" library="rcl" deviceset="R-US_" device="R0402" value="4.75k">
+<attribute name="DIGIKEY" value="RHM1.00MCDCT-ND"/>
+</part>
+<part name="R9" library="rcl" deviceset="R-US_" device="R0402" value="5.6k 5%">
+<attribute name="DIGIKEY" value="RHM1.00MCDCT-ND"/>
+</part>
+<part name="R10" library="rcl" deviceset="R-US_" device="R0402" value="5.6k 5%">
+<attribute name="DIGIKEY" value="RHM1.00MCDCT-ND"/>
+</part>
+<part name="R11" library="rcl" deviceset="R-US_" device="R0402" value="10k 1%">
+<attribute name="DIGIKEY" value="RHM1.00MCDCT-ND"/>
+</part>
 </parts>
 <sheets>
@@
 <instance part="SUPPLY2" gate="G$1" x="99.06" y="35.56"/>
 <instance part="SJ1" gate="G$1" x="15.24" y="12.7"/>
-<instance part="R8" gate="G$1" x="25.4" y="40.64" rot="R90"/>
-<instance part="R7" gate="G$1" x="33.02" y="40.64" rot="R90"/>
-<instance part="R6" gate="G$1" x="40.64" y="40.64" rot="R90"/>
-<instance part="R9" gate="G$1" x="17.78" y="40.64" rot="R90"/>
-<instance part="R10" gate="G$1" x="10.16" y="40.64" rot="R90"/>
-<instance part="R11" gate="G$1" x="86.36" y="17.78" rot="R180"/>
 <instance part="WRT" gate="G$1" x="78.74" y="10.16" rot="R270"/>
 <instance part="GND9" gate="1" x="71.12" y="5.08"/>
+<instance part="R6" gate="G$1" x="40.64" y="40.64" rot="R90">
+<attribute name="DIGIKEY" x="40.64" y="40.64" size="1.27" layer="96" rot="R90" display="off"/>
+</instance>
+<instance part="R7" gate="G$1" x="33.02" y="40.64" rot="R90">
+<attribute name="DIGIKEY" x="33.02" y="40.64" size="1.27" layer="96" rot="R90" display="off"/>
+</instance>
+<instance part="R8" gate="G$1" x="25.4" y="40.64" rot="R90">
+<attribute name="DIGIKEY" x="25.4" y="40.64" size="1.27" layer="96" rot="R90" display="off"/>
+</instance>
+<instance part="R9" gate="G$1" x="17.78" y="40.64" rot="R90">
+<attribute name="DIGIKEY" x="17.78" y="40.64" size="1.27" layer="96" rot="R90" display="off"/>
+</instance>
+<instance part="R10" gate="G$1" x="10.16" y="40.64" rot="R90">
+<attribute name="DIGIKEY" x="10.16" y="40.64" size="1.27" layer="96" rot="R90" display="off"/>
+</instance>
+<instance part="R11" gate="G$1" x="86.36" y="17.78" rot="R180">
+<attribute name="DIGIKEY" x="86.36" y="17.78" size="1.27" layer="96" rot="R180" display="off"/>
+</instance>
 </instances>
 <busses>
@@
 </segment>
 <segment>
-<pinref part="R10" gate="G$1" pin="2"/>
 <pinref part="SUPPLY1" gate="G$1" pin="VCC"/>
 <wire x1="10.16" y1="45.72" x2="10.16" y2="50.8" width="0.2032" layer="91"/>
-<pinref part="R8" gate="G$1" pin="2"/>
 <wire x1="10.16" y1="50.8" x2="10.16" y2="53.34" width="0.2032" layer="91"/>
 <wire x1="25.4" y1="45.72" x2="25.4" y2="50.8" width="0.2032" layer="91"/>
-<pinref part="R7" gate="G$1" pin="2"/>
 <wire x1="33.02" y1="45.72" x2="33.02" y2="50.8" width="0.2032" layer="91"/>
-<pinref part="R6" gate="G$1" pin="2"/>
 <wire x1="33.02" y1="50.8" x2="40.64" y2="50.8" width="0.2032" layer="91"/>
 <wire x1="40.64" y1="50.8" x2="40.64" y2="45.72" width="0.2032" layer="91"/>
@@
 <junction x="25.4" y="50.8"/>
 <wire x1="25.4" y1="50.8" x2="17.78" y2="50.8" width="0.2032" layer="91"/>
-<pinref part="R9" gate="G$1" pin="2"/>
 <wire x1="10.16" y1="50.8" x2="17.78" y2="50.8" width="0.2032" layer="91"/>
 <wire x1="17.78" y1="50.8" x2="17.78" y2="45.72" width="0.2032" layer="91"/>
 <junction x="17.78" y="50.8"/>
 <junction x="10.16" y="50.8"/>
+<pinref part="R6" gate="G$1" pin="2"/>
+<pinref part="R7" gate="G$1" pin="2"/>
+<pinref part="R8" gate="G$1" pin="2"/>
+<pinref part="R9" gate="G$1" pin="2"/>
+<pinref part="R10" gate="G$1" pin="2"/>
 </segment>
 <segment>
@@
 <wire x1="99.06" y1="33.02" x2="99.06" y2="35.56" width="0.2032" layer="91"/>
 <pinref part="SUPPLY2" gate="G$1" pin="VCC"/>
-<pinref part="R11" gate="G$1" pin="1"/>
 <wire x1="91.44" y1="17.78" x2="93.98" y2="17.78" width="0.2032" layer="91"/>
 <wire x1="93.98" y1="17.78" x2="93.98" y2="33.02" width="0.2032" layer="91"/>
 <junction x="93.98" y="33.02"/>
 <junction x="99.06" y="33.02"/>
+<pinref part="R11" gate="G$1" pin="1"/>
 </segment>
 </net>
@@
 <pinref part="U2" gate="G$1" pin="A0"/>
 <wire x1="15.24" y1="22.86" x2="40.64" y2="22.86" width="0.2032" layer="91"/>
-<pinref part="R6" gate="G$1" pin="1"/>
 <wire x1="40.64" y1="22.86" x2="43.18" y2="22.86" width="0.2032" layer="91"/>
 <wire x1="40.64" y1="35.56" x2="40.64" y2="22.86" width="0.2032" layer="91"/>
 <junction x="40.64" y="22.86"/>
+<pinref part="R6" gate="G$1" pin="1"/>
 </segment>
 </net>
@@
 <pinref part="SJ1" gate="G$1" pin="3"/>
 <wire x1="22.86" y1="7.62" x2="15.24" y2="7.62" width="0.2032" layer="91"/>
-<pinref part="R7" gate="G$1" pin="1"/>
 <wire x1="33.02" y1="35.56" x2="33.02" y2="20.32" width="0.2032" layer="91"/>
 <junction x="33.02" y="20.32"/>
+<pinref part="R7" gate="G$1" pin="1"/>
 </segment>
 </net>
@@
 <pinref part="U2" gate="G$1" pin="A2"/>
 <wire x1="43.18" y1="17.78" x2="25.4" y2="17.78" width="0.2032" layer="91"/>
+<wire x1="25.4" y1="35.56" x2="25.4" y2="17.78" width="0.2032" layer="91"/>
 <pinref part="R8" gate="G$1" pin="1"/>
-<wire x1="25.4" y1="35.56" x2="25.4" y2="17.78" width="0.2032" layer="91"/>
 </segment>
 </net>
@@
 <segment>
 <pinref part="U2" gate="G$1" pin="SDA"/>
-<pinref part="R10" gate="G$1" pin="1"/>
 <wire x1="43.18" y1="27.94" x2="10.16" y2="27.94" width="0.2032" layer="91"/>
 <wire x1="10.16" y1="27.94" x2="10.16" y2="35.56" width="0.2032" layer="91"/>
@@
 <junction x="10.16" y="27.94"/>
 <label x="7.62" y="27.94" size="1.27" layer="95" rot="R180" xref="yes"/>
+<pinref part="R10" gate="G$1" pin="1"/>
 </segment>
 <segment>
@@
 <pinref part="U2" gate="G$1" pin="SCL"/>
 <wire x1="43.18" y1="33.02" x2="17.78" y2="33.02" width="0.2032" layer="91"/>
-<pinref part="R9" gate="G$1" pin="1"/>
 <wire x1="17.78" y1="33.02" x2="7.62" y2="33.02" width="0.2032" layer="91"/>
 <wire x1="17.78" y1="35.56" x2="17.78" y2="33.02" width="0.2032" layer="91"/>
 <junction x="17.78" y="33.02"/>
 <label x="7.62" y="33.02" size="1.27" layer="95" rot="R180" xref="yes"/>
+<pinref part="R9" gate="G$1" pin="1"/>
 </segment>
 <segment>
@@
 <segment>
 <pinref part="U2" gate="G$1" pin="WP"/>
-<pinref part="R11" gate="G$1" pin="2"/>
 <wire x1="71.12" y1="17.78" x2="73.66" y2="17.78" width="0.2032" layer="91"/>
 <wire x1="73.66" y1="17.78" x2="81.28" y2="17.78" width="0.2032" layer="91"/>
@@
 <pinref part="WRT" gate="G$1" pin="1"/>
 <wire x1="76.2" y1="10.16" x2="73.66" y2="10.16" width="0.2032" layer="91"/>
-</segment>
-</net>
+<pinref part="R11" gate="G$1" pin="2"/>
+</segment>
+</net>

Commit message: fixed labeling and vias
Parts:
- removed C26: 6.8pF, rcl:C-EUC0402
- removed L12: 1nH, SparkFun-Passives:INDUCTOR0402
- removed U5: CC2520, chips:CC2520
- added C22: 100nF, rcl:C-EUC0402
- added U3: CAT24C256WI-GT3, bbb-cc2520:CAT24C256WI-GT3
- C1: value 100nF -> 1pF
- C10, C8, C9: value 100nF -> 27pF; DIGIKEY 490-1318-1-ND -> 490-5869-1-ND
- C11, C13: value 100nF -> 1nF
- C12: value 1uF -> 1nF; device rcl:C-EUC0603 -> rcl:C-EUC0402; DIGIKEY 490-1550-1-ND -> 490-1318-1-ND
- C14, C15: value 27pF -> 100nF; DIGIKEY 490-5869-1-ND -> 490-1318-1-ND
- C16: value 3pF -> 100nF
- C17: value 3.9pF -> 100nF
- C18, C19, C21: value 1nF -> 100nF
- C2: value 100nF -> 2.7pF
- C20: value 15pF -> 100nF
- C23: value 2.2uF -> 1uF; device rcl:C-EUC0402 -> rcl:C-EUC0603; DIGIKEY 490-1318-1-ND -> 490-1550-1-ND
- C24: value 2.7pF -> 1uF; device rcl:C-EUC0402 -> rcl:C-EUC0603; DIGIKEY 490-1318-1-ND -> 490-1550-1-ND
- C25: value 1pF -> 2.2uF
- C3: value 100nF -> 3pF
- C4: value 1uF -> 6.8pF; device rcl:C-EUC0603 -> rcl:C-EUC0402; DIGIKEY 490-1550-1-ND -> 490-1318-1-ND
- C5: value 100nF -> 15pF
- C6: value 27pF -> 3.9pF; DIGIKEY 490-5869-1-ND -> 490-1318-1-ND
- L10: value 1kOhm -> 5.1nH
- L11: value 1.5nH -> 1kOhm
- L4: value 2nH -> 1nH
- L7: value (none) -> 1.1nH
- L8: value 1.1nH -> 1.5nH
- L9: value 5.1nH -> 2nH
- R11: value 10k 1% -> 5.6k 5%
- R12: value 1M 1% -> 10k 1%
- R14: value 4.3k -> 56k 1%
- R15: value 1k 1% -> 330k 1%
- R16: value 1k 1% -> 1M 1%; DIGIKEY P56.0KLCT-ND -> RHM1.00MCDCT-ND
- R17: value 330k 1% -> 1M 1%; DIGIKEY P56.0KLCT-ND -> RHM1.00MCDCT-ND
- R4: value 1M 1% -> 1k 1%; DIGIKEY RHM1.00MCDCT-ND -> P56.0KLCT-ND
- R5: value 56k 1% -> 1k 1%
- R6: value 4.75k -> 4.3k; DIGIKEY RHM1.00MCDCT-ND -> P56.0KLCT-ND
- R9: value 5.6k 5% -> 4.75k
- U2: value CAT24C256WI-GT3 -> CC2520; device bbb-cc2520:CAT24C256WI-GT3 -> chips:CC2520
Connections:
- net !RESET1: now also U2.!RESET; no longer U5.!RESET
- net CCA1: now also U2.GPIO3; no longer U5.GPIO3
- net CS1: now also U2.!CS; no longer U5.!CS
- net EN: now also R5.2, U2.GPIO0; no longer R16.2, U5.GPIO0
- net FIFO1: now also U2.GPIO1; no longer U5.GPIO1
- net FIFOP1: now also U2.GPIO2; no longer U5.GPIO2
- net GND: now also C16.2, C17.2, C22.2, L3.1, L4.1, L6.2, R16.1, R17.1, R6.1, U2.GND_EXP, U3.VSS; no longer C3.2, C4.2, C6.2, L12.2, L5.1, L6.1, R12.1, R4.1, R5.1, U2.VSS, U5.GND_EXP
- net MISO: now also R16.2, R17.2, U2.MISO; no longer R12.2, R4.2, U5.MISO
- net MOSI: now also U2.MOSI; no longer U5.MOSI
- net N$11: now also C8.1; no longer C7.1
- net N$12: now also C17.1; no longer C5.1
- net N$13: now also C7.1; no longer C6.1
- net N$14: now also R13.2; no longer R5.2
- net N$29: now also R7.1, U3.A0; no longer R6.1, U2.A0
- net N$30: now also R8.1, U3.A1; no longer R7.1, U2.A1
- net N$31: now also R12.2, U3.WP; no longer R11.2, U2.WP
- net N$32: now also R9.1, U3.A2; no longer R8.1, U2.A2
- net N$44: now also L9.1; no longer L4.1, L7.1
- net N$45: now also L5.1; no longer L3.1, L7.2
- net N$46: now also C6.2, L4.2, L5.2; no longer C17.2, L3.2, L6.2
- net N$47: now also C3.2, L3.2, L9.2; no longer C16.2, L4.2, L5.2
- net N$48: now also L10.1, L7.1; no longer L8.1, L9.1
- net N$49: now also C11.1, C12.1, C13.1, C25.1, L11.2; no longer C18.1, C19.1, C21.1, C23.1, L9.2
- net N$5: now also C14.1, C15.1, C16.1, C23.1; no longer C1.1, C2.1, C3.1, C4.1
- net N$50: now also C5.1, L7.2; no longer C20.1, L8.2
- net N$51: now also L8.2; no longer L11.2
- net N$52: now also C2.1, C4.1, L6.1; no longer C24.1, C26.1, L12.1
- net N$53: now also C1.1, C4.2, L8.1; no longer C25.1, C26.2, L11.1
- net N$54: now also R6.2; no longer R14.2
- net N$55: now also R4.1; no longer R15.1
- net N$56: now also R5.1; no longer R16.1
- net N$57: now also C19.1, C20.1, C21.1, C24.1, U2.AVDD0, U2.AVDD1, U2.AVDD2, U2.AVDD3, U2.AVDD4, U2.AVDD5, U2.DVDD, U2.VREG_EN; no longer C10.1, C11.1, C12.1, C9.1, U5.AVDD0, U5.AVDD1, U5.AVDD2, U5.AVDD3, U5.AVDD4, U5.AVDD5, U5.DVDD, U5.VREG_EN
- net N$58: now also C22.1, U2.DCOUPL; no longer C13.1, U5.DCOUPL
- net N$59: now also C10.1, U2.XOSC_Q1; no longer C15.1, U5.XOSC_Q1
- net N$60: now also C9.1, U2.XOSC_Q2; no longer C14.1, U5.XOSC_Q2
- net N$61: now also R14.2, U2.RBIAS; no longer R13.2, U5.RBIAS
- net N$62: now also R15.1; no longer R17.1
- net PAEN: now also R4.2, U2.GPIO5; no longer R15.2, U5.GPIO5
- net RF_N2: now also C6.1, U2.RF_N; no longer C17.1, U5.RF_N
- net RF_P2: now also C3.1, U2.RF_P; no longer C16.1, U5.RF_P
- net SCL: now also R10.1, U3.SCL; no longer R9.1, U2.SCL
- net SCLK: now also U2.SCLK; no longer U5.SCLK
- net SDA: now also R11.1, U3.SDA; no longer R10.1, U2.SDA
- net SFD1: now also U2.GPIO4; no longer U5.GPIO4
- net VCC: now also C18.1, L11.1, R11.2, R12.1, R15.2, U3.VCC; no longer C8.1, L10.1, R11.1, R17.2, R6.2, U2.VCC
Other:
- moved on the sheet: C10, C11, C12, C13, C19, C20, C21, C24, C25, C7, C8, C9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

Commit message: rev a finished, gerbers generated, bom done
Parts:
- removed U$1: UMICH_SOLID_SMALL, logos:UMICH_SOLID_SMALL
- renumbered IC1 to U4
Changed lines of the file:
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@@
 <parts>
 <part name="FRAME1" library="frames" deviceset="LETTER_L" device=""/>
-<part name="U$1" library="logos" deviceset="UMICH_SOLID" device="_SMALL"/>
 <part name="D1" library="SparkFun-LED" deviceset="LED" device="0603">
 <attribute name="DIGIKEY" value="160-1834-1-ND"/>
@@
 <part name="P+12" library="SparkFun" deviceset="VCC" device=""/>
 <part name="GND42" library="supply1" deviceset="GND" device=""/>
-<part name="IC1" library="bbb-cc2520" deviceset="CC2591" device=""/>
+<part name="U4" library="bbb-cc2520" deviceset="CC2591" device=""/>
 <part name="L5" library="SparkFun-Passives" deviceset="INDUCTOR" device="0402" value="1nH"/>
 <part name="L9" library="SparkFun-Passives" deviceset="INDUCTOR" device="0402" value="2nH"/>
@@
 <instance part="FRAME1" gate="G$1" x="0" y="0"/>
 <instance part="FRAME1" gate="G$2" x="147.32" y="0"/>
-<instance part="U$1" gate="G$1" x="231.14" y="172.72"/>
 <instance part="D1" gate="G$1" x="218.44" y="86.36">
 <attribute name="DIGIKEY" x="218.44" y="86.36" size="1.27" layer="96" display="off"/>
@@
 <instance part="P+12" gate="1" x="58.42" y="165.1"/>
 <instance part="GND42" gate="1" x="111.76" y="73.66"/>
-<instance part="IC1" gate="G$1" x="180.34" y="60.96"/>
+<instance part="U4" gate="G$1" x="180.34" y="60.96"/>
 <instance part="L5" gate="G$1" x="132.08" y="60.96" rot="R270"/>
 <instance part="L9" gate="G$1" x="132.08" y="83.82" rot="R270"/>
@@
 </segment>
 <segment>
-<pinref part="IC1" gate="G$1" pin="GND@1"/>
+<pinref part="U4" gate="G$1" pin="GND@1"/>
 <wire x1="198.12" y1="50.8" x2="208.28" y2="50.8" width="0.1524" layer="91"/>
 <wire x1="208.28" y1="50.8" x2="208.28" y2="48.26" width="0.1524" layer="91"/>
-<pinref part="IC1" gate="G$1" pin="GND@2"/>
+<pinref part="U4" gate="G$1" pin="GND@2"/>
 <wire x1="208.28" y1="48.26" x2="198.12" y2="48.26" width="0.1524" layer="91"/>
-<pinref part="IC1" gate="G$1" pin="GND@3"/>
+<pinref part="U4" gate="G$1" pin="GND@3"/>
 <wire x1="198.12" y1="45.72" x2="208.28" y2="45.72" width="0.1524" layer="91"/>
 <wire x1="208.28" y1="45.72" x2="208.28" y2="48.26" width="0.1524" layer="91"/>
-<pinref part="IC1" gate="G$1" pin="GND@4"/>
+<pinref part="U4" gate="G$1" pin="GND@4"/>
 <wire x1="198.12" y1="43.18" x2="208.28" y2="43.18" width="0.1524" layer="91"/>
 <wire x1="208.28" y1="43.18" x2="208.28" y2="45.72" width="0.1524" layer="91"/>
-<pinref part="IC1" gate="G$1" pin="GND@5"/>
+<pinref part="U4" gate="G$1" pin="GND@5"/>
 <wire x1="198.12" y1="40.64" x2="208.28" y2="40.64" width="0.1524" layer="91"/>
 <wire x1="208.28" y1="40.64" x2="208.28" y2="43.18" width="0.1524" layer="91"/>
@@
 <net name="N$44" class="0">
 <segment>
-<pinref part="IC1" gate="G$1" pin="RF_P"/>
+<pinref part="U4" gate="G$1" pin="RF_P"/>
 <wire x1="162.56" y1="76.2" x2="160.02" y2="76.2" width="0.1524" layer="91"/>
 <wire x1="160.02" y1="76.2" x2="160.02" y2="83.82" width="0.1524" layer="91"/>
@@
 <net name="N$45" class="0">
 <segment>
-<pinref part="IC1" gate="G$1" pin="RF_N"/>
+<pinref part="U4" gate="G$1" pin="RF_N"/>
 <wire x1="162.56" y1="66.04" x2="160.02" y2="66.04" width="0.1524" layer="91"/>
 <wire x1="160.02" y1="66.04" x2="160.02" y2="60.96" width="0.1524" layer="91"/>
@@
 <net name="N$49" class="0">
 <segment>
-<pinref part="IC1" gate="G$1" pin="AVDD_PA1"/>
+<pinref part="U4" gate="G$1" pin="AVDD_PA1"/>
 <wire x1="198.12" y1="73.66" x2="208.28" y2="73.66" width="0.1524" layer="91"/>
 <wire x1="208.28" y1="73.66" x2="208.28" y2="124.46" width="0.1524" layer="91"/>
@@
 <junction x="187.96" y="124.46"/>
 <wire x1="208.28" y1="124.46" x2="187.96" y2="124.46" width="0.1524" layer="91"/>
-<pinref part="IC1" gate="G$1" pin="AVDD_BIAS"/>
+<pinref part="U4" gate="G$1" pin="AVDD_BIAS"/>
 <wire x1="198.12" y1="76.2" x2="205.74" y2="76.2" width="0.1524" layer="91"/>
 <wire x1="205.74" y1="76.2" x2="205.74" y2="104.14" width="0.1524" layer="91"/>
@@
 <wire x1="187.96" y1="124.46" x2="157.48" y2="124.46" width="0.1524" layer="91"/>
 <junction x="157.48" y="124.46"/>
-<pinref part="IC1" gate="G$1" pin="AVDD_LNA"/>
+<pinref part="U4" gate="G$1" pin="AVDD_LNA"/>
 <wire x1="198.12" y1="68.58" x2="213.36" y2="68.58" width="0.1524" layer="91"/>
 <wire x1="213.36" y1="68.58" x2="213.36" y2="170.18" width="0.1524" layer="91"/>
@@
 <net name="N$48" class="0">
 <segment>
-<pinref part="IC1" gate="G$1" pin="AVDD_PA2"/>
+<pinref part="U4" gate="G$1" pin="AVDD_PA2"/>
 <wire x1="198.12" y1="71.12" x2="210.82" y2="71.12" width="0.1524" layer="91"/>
 <wire x1="210.82" y1="71.12" x2="210.82" y2="142.24" width="0.1524" layer="91"/>
@@
 <net name="N$51" class="0">
 <segment>
-<pinref part="IC1" gate="G$1" pin="ANT"/>
+<pinref part="U4" gate="G$1" pin="ANT"/>
 <pinref part="L8" gate="G$1" pin="2"/>
 <wire x1="198.12" y1="60.96" x2="215.9" y2="60.96" width="0.1524" layer="91"/>
@@
 <net name="N$54" class="0">
 <segment>
-<pinref part="IC1" gate="G$1" pin="BIAS"/>
+<pinref part="U4" gate="G$1" pin="BIAS"/>
 <pinref part="R6" gate="G$1" pin="2"/>
 <wire x1="198.12" y1="55.88" x2="218.44" y2="55.88" width="0.1524" layer="91"/>
@@
 <segment>
 <pinref part="R4" gate="G$1" pin="1"/>
-<pinref part="IC1" gate="G$1" pin="PAEN"/>
+<pinref part="U4" gate="G$1" pin="PAEN"/>
 <wire x1="160.02" y1="55.88" x2="162.56" y2="55.88" width="0.1524" layer="91"/>
 </segment>
@@
 <segment>
 <pinref part="R5" gate="G$1" pin="1"/>
-<pinref part="IC1" gate="G$1" pin="EN"/>
+<pinref part="U4" gate="G$1" pin="EN"/>
 <wire x1="160.02" y1="48.26" x2="162.56" y2="48.26" width="0.1524" layer="91"/>
 </segment>
@@
 <net name="N$62" class="0">
 <segment>
-<pinref part="IC1" gate="G$1" pin="HGM"/>
+<pinref part="U4" gate="G$1" pin="HGM"/>
 <pinref part="R15" gate="G$1" pin="1"/>
 <wire x1="162.56" y1="40.64" x2="160.02" y2="40.64" width="0.1524" layer="91"/>
