File: hardware/eagle/bbb-cc2520/rev_b/bbb-cc2520_b.sch (EAGLE design)
At the start: 68 parts, among them P1 MOLEX_73251-135X, P2 MOLEX_73251-135X, P9/P8 BBB_HEADERS, U1 CC2520, U2 CC2520, U3 CAT24C256WI-GT3, U4 CC2591, X1 NX2520SA, X2 NX2520SA

Commit message: revb mostly finished, need to add BLE chip
Parts:
- added R18, R19: 10k 1%, rcl:R-US_R0402
- added U5: CD4051B-53B, bbb-cc2520:CD4051B-53B
Connections:
- new net CS: P9/P8.I2C1_SCL, U5.COM
- new net CS2: U5.2
- new net CS3: U5.3
- new net CS4: U5.4
- new net CS5: U5.5
- new net CS6: U5.6
- new net CS7: U5.7
- new net SPIE0: P9/P8.GPIO1_13, U5.A
- new net SPIE1: P9/P8.GPIO1_12, U5.B
- new net SPIE2: U5.C
- net !RESET0: now also P9/P8.GPIO1_28; no longer P9/P8.GPIO1_16
- net CCA0: now also P9/P8.GPIO1_16; no longer P9/P8.GPIO1_28
- net CCA1: now also P9/P8.GPIO0_26; no longer P9/P8.GPIO1_12
- net CS0: now also R18.1, U5.0; no longer P9/P8.I2C1_SCL
- net CS1: now also R19.1, U5.1; no longer P9/P8.EHRPWM1B
- net FIFO1: now also P9/P8.GPIO1_14; no longer P9/P8.GPIO0_26
- net FIFOP1: now also P9/P8.EHRPWM2B; no longer P9/P8.GPIO1_13
- net GND: now also U5.INH, U5.VEE, U5.VSS
- net LED0: now also P9/P8.EHRPWM2A; no longer P9/P8.GPIO0_27
- net LED1: now also P9/P8.GPIO0_27; no longer P9/P8.GPIO2_1
- net LED2: now also P9/P8.GPIO2_1; no longer P9/P8.GPIO1_14
- net MISO: now also P9/P8.UART2_TXD; no longer P9/P8.I2C1_SDA
- net MOSI: now also P9/P8.I2C1_SDA; no longer P9/P8.UART2_TXD
- net VCC: now also R18.2, R19.2, U5.VDD

Commit message: RevB finished
Parts:
- removed P1, P2: MOLEX_73251-135X, connector:MOLEX_73251-135X
- added ANT1, ANT2, ANT3: MOLEX_WM5544-ND, connector:MOLEX_WM5544-ND
- added B2: BAL-NRF01D3, chips:BAL-NRF01D3
- added C26: 0.1uF, passives:CAPACITOR
- added C27, C32: 1nF, passives:CAPACITOR
- added C28: 4.7uF, passives:CAPACITOR
- added C29: 1uF, passives:CAPACITOR
- added C30, C31: 12pF, passives:CAPACITOR
- added C33: 47nF, passives:CAPACITOR
- added C34: 2.2nF, passives:CAPACITOR
- added C35: 0.8pF, passives:CAPACITOR
- added D4: BLUE, SparkFun-LED:LED0603
- added J1: TC2030-IDC, connector:TC2030-IDC
- added JP1: (no value), jumper:JP2Q
- added L12: (no value), passives:INDUCTOR0402
- added L13: 10uH, passives:INDUCTOR0603
- added R20, R21: 10k 1%, rcl:R-US_R0402
- added R22: 470, rcl:R-US_R0402
- added R23: 12k, passives:RESISTOR
- added U6: NRF51822QF, chips:NRF51822QF
- added X3: 16MHz, crystals:TXC-8Y
Connections:
- removed net SPIE2: U5.C
- new net A0: U6.P26/AIN0/XL2
- new net A1: U6.P27/AIN1/XL1
- new net AVDD: C27.1, C29.1, L12.1, U6.AVDD
- new net BIRQ: P9/P8.EHRPWM1B, U6.P07
- new net DCC: L13.2, U6.DCC
- new net N$36: B2.ANT1, U6.ANT1
- new net N$37: B2.ANT2, U6.ANT2
- new net N$38: ANT3.P$1, B2.SE, C35.1
- new net N$39: L12.2, L13.1
- new net N$40: C30.1, U6.XC1, X3.1
- new net N$41: C31.1, U6.XC2, X3.2
- new net N$42: C32.1, U6.DEC1
- new net N$43: C33.1, U6.DEC2
- new net N$63: D4.A, R22.1
- new net N$64: R22.2, U6.P13
- new net P03: JP1.1, U6.P03/AIN4
- new net P04: JP1.2, U6.P04/AIN5
- new net P05: JP1.4, U6.P05/AIN6
- new net P06: JP1.3, U6.P06/AIN7/AREF1
- new net P12: U6.P12
- new net P24: U6.P24
- new net P25: U6.P25
- new net PROG_RX: U6.P28
- new net PROG_TX: U6.P29
- new net SWDCLK: J1.4, R23.1, U6.SWDCLK
- new net SWDIO: J1.2, U6.SWDIO/!RESET
- new net VDD_PA: B2.VDD_PA, C34.1, U6.VDD_PA
- net CS0: now also R19.1; no longer R18.1
- net CS1: now also R20.1; no longer R19.1
- net CS2: now also R21.1, U6.P11
- net CS4: now also R18.1
- net GND: now also ANT1.P$2, ANT1.P$3, ANT1.P$4, ANT1.P$5, ANT2.P$2, ANT2.P$3, ANT2.P$4, ANT2.P$5, ANT3.P$2, ANT3.P$3, ANT3.P$4, ANT3.P$5, B2.GND, C26.2, C27.2, C28.2, C29.2, C30.2, C31.2, C32.2, C33.2, C34.2, C35.2, D4.C, J1.5, R23.2, U5.C, U6.GND; no longer P1.P$2, P1.P$3, P1.P$4, P1.P$5, P2.P$2, P2.P$3, P2.P$4, P2.P$5, P9/P8.GND6
- net MISO: now also U6.P09
- net MOSI: now also U6.P08
- net N$52: now also ANT2.P$1; no longer P2.P$1
- net N$7: now also ANT1.P$1; no longer P1.P$1
- net SCLK: now also U6.P10
- net VCC: now also C26.1, C28.1, J1.1, R20.2, R21.2, U6.VDD
Other:
- note added: "PIN1"
- note added: "PIN12"
- note added: "PIN36"
- moved on the sheet: R18, R19, U5

Commit message: added label for bluetooth irq
Connections:
- net SPIE0 renamed CSE0
- net SPIE1 renamed CSE1
Changed lines of the file:
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@@
 <setting verticaltext="up"/>
 </settings>
-<grid distance="0.1" unitdist="inch" unit="inch" style="lines" multiple="1" display="no" altdistance="0.01" altunitdist="inch" altunit="inch"/>
+<grid distance="0.1" unitdist="inch" unit="inch" style="lines" multiple="1" display="yes" altdistance="0.01" altunitdist="inch" altunit="inch"/>
 <layers>
 <layer number="1" name="Top" color="4" fill="1" visible="no" active="no"/>
@@
 </segment>
 </net>
-<net name="SPIE0" class="0">
+<net name="CSE0" class="0">
 <segment>
 <pinref part="P9/P8" gate="G$1" pin="GPIO1_13"/>
@@
 </segment>
 </net>
-<net name="SPIE1" class="0">
+<net name="CSE1" class="0">
 <segment>
 <pinref part="P9/P8" gate="G$1" pin="GPIO1_12"/>
@@
 </segment>
 </net>
-<net name="SPIE0" class="0">
-<segment>
-<pinref part="U5" gate="G$1" pin="A"/>
-<wire x1="195.58" y1="129.54" x2="198.12" y2="129.54" width="0.1524" layer="91"/>
-<label x="198.12" y="129.54" size="1.27" layer="95" xref="yes"/>
-</segment>
-</net>
 <net name="CS0" class="0">
 <segment>
@@
 <wire x1="195.58" y1="134.62" x2="198.12" y2="134.62" width="0.1524" layer="91"/>
 <label x="198.12" y="134.62" size="1.27" layer="95" xref="yes"/>
-</segment>
-</net>
-<net name="SPIE1" class="0">
-<segment>
-<pinref part="U5" gate="G$1" pin="B"/>
-<wire x1="195.58" y1="124.46" x2="198.12" y2="124.46" width="0.1524" layer="91"/>
-<label x="198.12" y="124.46" size="1.27" layer="95" xref="yes"/>
 </segment>
 </net>
@@
 </segment>
 </net>
+<net name="CSE0" class="0">
+<segment>
+<pinref part="U5" gate="G$1" pin="A"/>
+<wire x1="195.58" y1="129.54" x2="198.12" y2="129.54" width="0.1524" layer="91"/>
+<label x="198.12" y="129.54" size="1.27" layer="95" xref="yes"/>
+</segment>
+</net>
+<net name="CSE1" class="0">
+<segment>
+<pinref part="U5" gate="G$1" pin="B"/>
+<wire x1="195.58" y1="124.46" x2="198.12" y2="124.46" width="0.1524" layer="91"/>
+<label x="198.12" y="124.46" size="1.27" layer="95" xref="yes"/>
+</segment>
+</net>

Commit message: updated symbol for demux, added test points
Parts:
- removed R18: 10k 1%, rcl:R-US_R0402
- added CS0, CS1, CS2: TEST_POINT_0.040IN, headers:TEST_POINT_0.040IN
Connections:
- removed net CS3: U5.3
- removed net CS4: R18.1, U5.4
- removed net CS5: U5.5
- removed net CS6: U5.6
- removed net CS7: U5.7
- net CS0: now also CS0.TESTPOINT
- net CS1: now also CS1.TESTPOINT
- net CS2: now also CS2.TESTPOINT
- net VCC: no longer R18.2

Commit message: made changes to board in regards to issue 3
Parts:
- removed JP1: (no value), jumper:JP2Q
- added CS3, CS4: TPTP14SQ, testpad:TPTP14SQ
- added SJ2: JUMPER-PAD-2-NC_BY_TRACE, SparkFun-Passives:JUMPER-PAD-2-NC_BY_TRACE
Connections:
- removed net P04: JP1.2, U6.P04/AIN5
- removed net P05: JP1.4, U6.P05/AIN6
- removed net P06: JP1.3, U6.P06/AIN7/AREF1
- new net !RESET2: P9/P8.UART4_RXD, U6.P04/AIN5
- new net N$65: SJ2.1, U5.C
- new net N$66: CS3.TP, U5.3
- new net N$67: CS4.TP, U5.4
- new net UARTRX: P9/P8.UART1_TXD, U6.P05/AIN6
- new net UARTTX: P9/P8.UART1_RXD, U6.P06/AIN7/AREF1
- net GND: now also SJ2.2; no longer U5.C
- net P03: no longer JP1.1
Other:
- moved on the sheet: CS0, CS1, CS2
Changed lines of the file:
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@@
 <attribute name="DIGIKEY" value="RHM1.00MCDCT-ND"/>
 </part>
-<part name="JP1" library="jumper" deviceset="JP2Q" device=""/>
 <part name="R22" library="rcl" deviceset="R-US_" device="R0402" value="470">
 <attribute name="DIGIKEY" value="RHM470JCT-ND"/>
@@
 <part name="CS1" library="headers" deviceset="TEST_POINT_0.040IN" device=""/>
 <part name="CS2" library="headers" deviceset="TEST_POINT_0.040IN" device=""/>
+<part name="SJ2" library="SparkFun-Passives" deviceset="JUMPER-PAD-2-NC_BY_TRACE" device=""/>
+<part name="CS4" library="testpad" deviceset="TP" device="TP14SQ"/>
+<part name="CS3" library="testpad" deviceset="TP" device="TP14SQ"/>
 </parts>
 <sheets>
@@
 <wire x1="121.92" y1="160.02" x2="127" y2="160.02" width="0.1524" layer="91"/>
 <label x="127" y="160.02" size="1.27" layer="95" xref="yes"/>
+</segment>
+</net>
+<net name="UARTRX" class="0">
+<segment>
+<pinref part="P9/P8" gate="G$1" pin="UART1_TXD"/>
+<wire x1="121.92" y1="149.86" x2="127" y2="149.86" width="0.1524" layer="91"/>
+<label x="127" y="149.86" size="1.27" layer="95" xref="yes"/>
+</segment>
+</net>
+<net name="UARTTX" class="0">
+<segment>
+<pinref part="P9/P8" gate="G$1" pin="UART1_RXD"/>
+<wire x1="121.92" y1="147.32" x2="127" y2="147.32" width="0.1524" layer="91"/>
+<label x="127" y="147.32" size="1.27" layer="95" xref="yes"/>
+</segment>
+</net>
+<net name="!RESET2" class="0">
+<segment>
+<pinref part="P9/P8" gate="G$1" pin="UART4_RXD"/>
+<label x="53.34" y="165.1" size="1.27" layer="95" rot="R180" xref="yes"/>
+<wire x1="58.42" y1="165.1" x2="53.34" y2="165.1" width="0.1524" layer="91"/>
 </segment>
 </net>
@@
 <instance part="P+13" gate="1" x="114.3" y="170.18"/>
 <instance part="GND54" gate="1" x="116.84" y="149.86"/>
-<instance part="JP1" gate="B1" x="63.5" y="170.18" rot="R270"/>
 <instance part="R22" gate="G$1" x="22.86" y="68.58" rot="R90">
 <attribute name="DIGIKEY" x="22.86" y="68.58" size="1.27" layer="96" rot="R90" display="off"/>
@@
 </segment>
 </net>
-<net name="P06" class="0">
+<net name="UARTTX" class="0">
 <segment>
 <pinref part="U6" gate="G$1" pin="P06/AIN7/AREF1"/>
@@
 <label x="48.26" y="88.9" size="1.27" layer="95" rot="R180" xref="yes"/>
 </segment>
-<segment>
-<pinref part="JP1" gate="B1" pin="3"/>
-<wire x1="55.88" y1="167.64" x2="53.34" y2="167.64" width="0.1524" layer="91"/>
-<label x="53.34" y="167.64" size="1.27" layer="95" rot="R180" xref="yes"/>
-</segment>
 </net>
 <net name="BIRQ" class="0">
@@
 </segment>
 </net>
-<net name="P05" class="0">
+<net name="UARTRX" class="0">
 <segment>
 <pinref part="U6" gate="G$1" pin="P05/AIN6"/>
@@
 <label x="48.26" y="91.44" size="1.27" layer="95" rot="R180" xref="yes"/>
 </segment>
-<segment>
-<pinref part="JP1" gate="B1" pin="4"/>
-<wire x1="71.12" y1="167.64" x2="73.66" y2="167.64" width="0.1524" layer="91"/>
-<label x="73.66" y="167.64" size="1.27" layer="95" xref="yes"/>
-</segment>
-</net>
-<net name="P04" class="0">
+</net>
+<net name="!RESET2" class="0">
 <segment>
 <pinref part="U6" gate="G$1" pin="P04/AIN5"/>
@@
 <label x="48.26" y="93.98" size="1.27" layer="95" rot="R180" xref="yes"/>
 </segment>
-<segment>
-<pinref part="JP1" gate="B1" pin="2"/>
-<wire x1="71.12" y1="170.18" x2="73.66" y2="170.18" width="0.1524" layer="91"/>
-<label x="73.66" y="170.18" size="1.27" layer="95" xref="yes"/>
-</segment>
 </net>
 <net name="P03" class="0">
-<segment>
-<pinref part="JP1" gate="B1" pin="1"/>
-<wire x1="53.34" y1="170.18" x2="55.88" y2="170.18" width="0.1524" layer="91"/>
-<label x="53.34" y="170.18" size="1.27" layer="95" rot="R180" xref="yes"/>
-</segment>
 <segment>
 <pinref part="U6" gate="G$1" pin="P03/AIN4"/>
@@
 <instance part="U5" gate="G$1" x="33.02" y="111.76"/>
 <instance part="P+7" gate="1" x="43.18" y="172.72"/>
-<instance part="GND18" gate="1" x="53.34" y="99.06"/>
+<instance part="GND18" gate="1" x="53.34" y="91.44"/>
 <instance part="R19" gate="G$1" x="71.12" y="160.02" rot="R90">
 <attribute name="DIGIKEY" x="71.12" y="160.02" size="1.27" layer="96" rot="R90" display="off"/>
@@
 <instance part="GND52" gate="1" x="55.88" y="167.64"/>
 <instance part="P+8" gate="1" x="71.12" y="172.72"/>
-<instance part="CS0" gate="G$1" x="71.12" y="134.62" rot="R90"/>
-<instance part="CS1" gate="G$1" x="78.74" y="134.62" rot="R90"/>
-<instance part="CS2" gate="G$1" x="86.36" y="134.62" rot="R90"/>
+<instance part="CS0" gate="G$1" x="71.12" y="124.46" rot="R90"/>
+<instance part="CS1" gate="G$1" x="78.74" y="124.46" rot="R90"/>
+<instance part="CS2" gate="G$1" x="86.36" y="124.46" rot="R90"/>
+<instance part="SJ2" gate="G$1" x="53.34" y="101.6" smashed="yes" rot="R270">
+<attribute name="NAME" x="55.88" y="104.14" size="1.778" layer="95" rot="R270"/>
+</instance>
+<instance part="CS4" gate="G$1" x="96.52" y="132.08" rot="R270"/>
+<instance part="CS3" gate="G$1" x="96.52" y="137.16" rot="R270"/>
 </instances>
 <busses>
@@
 <junction x="71.12" y="152.4"/>
 <pinref part="CS0" gate="G$1" pin="TESTPOINT"/>
-<wire x1="71.12" y1="152.4" x2="71.12" y2="137.16" width="0.1524" layer="91"/>
+<wire x1="71.12" y1="152.4" x2="71.12" y2="127" width="0.1524" layer="91"/>
 </segment>
 </net>
@@
 <junction x="78.74" y="147.32"/>
 <pinref part="CS1" gate="G$1" pin="TESTPOINT"/>
-<wire x1="78.74" y1="147.32" x2="78.74" y2="137.16" width="0.1524" layer="91"/>
+<wire x1="78.74" y1="147.32" x2="78.74" y2="127" width="0.1524" layer="91"/>
 </segment>
 </net>
@@
 <junction x="86.36" y="142.24"/>
 <pinref part="CS2" gate="G$1" pin="TESTPOINT"/>
-<wire x1="86.36" y1="142.24" x2="86.36" y2="137.16" width="0.1524" layer="91"/>
+<wire x1="86.36" y1="142.24" x2="86.36" y2="127" width="0.1524" layer="91"/>
 </segment>
 </net>
@@
 <segment>
 <pinref part="GND18" gate="1" pin="GND"/>
-<pinref part="U5" gate="G$1" pin="C"/>
-<wire x1="53.34" y1="101.6" x2="53.34" y2="107.95" width="0.1524" layer="91"/>
+<pinref part="SJ2" gate="G$1" pin="2"/>
+<wire x1="53.34" y1="93.98" x2="53.34" y2="96.52" width="0.1524" layer="91"/>
 </segment>
 </net>
@@
 </segment>
 </net>
+<net name="N$65" class="0">
+<segment>
+<pinref part="U5" gate="G$1" pin="C"/>
+<pinref part="SJ2" gate="G$1" pin="1"/>
+<wire x1="53.34" y1="107.95" x2="53.34" y2="106.68" width="0.1524" layer="91"/>
+</segment>
+</net>
+<net name="N$66" class="0">
+<segment>
+<pinref part="U5" gate="G$1" pin="3"/>
+<wire x1="63.5" y1="137.16" x2="93.98" y2="137.16" width="0.1524" layer="91"/>
+<pinref part="CS3" gate="G$1" pin="TP"/>
+</segment>
+</net>
+<net name="N$67" class="0">
+<segment>
+<pinref part="U5" gate="G$1" pin="4"/>
+<wire x1="63.5" y1="132.08" x2="93.98" y2="132.08" width="0.1524" layer="91"/>
+<pinref part="CS4" gate="G$1" pin="TP"/>
+</segment>
+</net>

Commit message: cleaned up pcb
Parts:
- renumbered WRT to J2
Connections:
- net GND: no longer D4.C
- net N$63: now also D4.C, R22.2; no longer D4.A, R22.1
- net N$64: now also R22.1; no longer R22.2
- net VCC: now also D4.A
Other:
- moved on the sheet: D4, R22
Changed lines of the file:
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@@
 <?xml version="1.0" encoding="utf-8"?>
 <!DOCTYPE eagle SYSTEM "eagle.dtd">
-<eagle version="6.6.0">
+<eagle version="6.5.0">
 <drawing>
 <settings>
@@
 <part name="SUPPLY2" library="SparkFun-Aesthetics" deviceset="VCC" device=""/>
 <part name="SJ1" library="SparkFun-Passives" deviceset="JUMPER-PAD-3-NO" device="FULL_BOX_SILK"/>
-<part name="WRT" library="SparkFun-Passives" deviceset="JUMPER-PTH-2-NO" device=""/>
+<part name="J2" library="SparkFun-Passives" deviceset="JUMPER-PTH-2-NO" device=""/>
 <part name="GND9" library="SparkFun-Aesthetics" deviceset="GND" device=""/>
 <part name="FRAME3" library="frames" deviceset="LETTER_L" device=""/>
@@
 <part name="GND49" library="supply1" deviceset="GND" device=""/>
 <part name="D4" library="SparkFun-LED" deviceset="LED" device="0603" value="BLUE"/>
-<part name="GND50" library="supply1" deviceset="GND" device=""/>
 <part name="L13" library="passives" deviceset="INDUCTOR" device="0603" value="10uH">
 <attribute name="DIGIKEY" value="490-4025-1-ND"/>
@@
 <part name="CS4" library="testpad" deviceset="TP" device="TP14SQ"/>
 <part name="CS3" library="testpad" deviceset="TP" device="TP14SQ"/>
+<part name="P+10" library="supply1" deviceset="VCC" device=""/>
 </parts>
 <sheets>
@@
 <instance part="SUPPLY2" gate="G$1" x="99.06" y="35.56"/>
 <instance part="SJ1" gate="G$1" x="15.24" y="12.7"/>
-<instance part="WRT" gate="G$1" x="78.74" y="10.16" rot="R270"/>
+<instance part="J2" gate="G$1" x="78.74" y="10.16" rot="R270"/>
 <instance part="GND9" gate="1" x="71.12" y="5.08"/>
 <instance part="R7" gate="G$1" x="40.64" y="40.64" rot="R90">
@@
 </segment>
 <segment>
-<pinref part="WRT" gate="G$1" pin="2"/>
+<pinref part="J2" gate="G$1" pin="2"/>
 <wire x1="76.2" y1="7.62" x2="71.12" y2="7.62" width="0.2032" layer="91"/>
 <pinref part="GND9" gate="1" pin="GND"/>
@@
 <wire x1="73.66" y1="17.78" x2="81.28" y2="17.78" width="0.2032" layer="91"/>
 <wire x1="73.66" y1="10.16" x2="73.66" y2="17.78" width="0.2032" layer="91"/>
-<pinref part="WRT" gate="G$1" pin="1"/>
+<pinref part="J2" gate="G$1" pin="1"/>
 <wire x1="76.2" y1="10.16" x2="73.66" y2="10.16" width="0.2032" layer="91"/>
 <pinref part="R12" gate="G$1" pin="2"/>
@@
 </instance>
 <instance part="GND49" gate="1" x="48.26" y="30.48"/>
-<instance part="D4" gate="G$1" x="22.86" y="58.42" smashed="yes">
-<attribute name="NAME" x="21.336" y="58.928" size="1.778" layer="95" rot="R90"/>
-<attribute name="VALUE" x="26.035" y="53.848" size="1.778" layer="96" rot="R90"/>
-</instance>
-<instance part="GND50" gate="1" x="22.86" y="48.26"/>
+<instance part="D4" gate="G$1" x="22.86" y="71.12" smashed="yes">
+<attribute name="NAME" x="21.336" y="71.628" size="1.778" layer="95" rot="R90"/>
+<attribute name="VALUE" x="26.035" y="66.548" size="1.778" layer="96" rot="R90"/>
+</instance>
 <instance part="L13" gate="G$1" x="33.02" y="119.38">
 <attribute name="DIGIKEY" x="33.02" y="119.38" size="1.778" layer="96" display="off"/>
@@
 <instance part="P+13" gate="1" x="114.3" y="170.18"/>
 <instance part="GND54" gate="1" x="116.84" y="149.86"/>
-<instance part="R22" gate="G$1" x="22.86" y="68.58" rot="R90">
-<attribute name="DIGIKEY" x="22.86" y="68.58" size="1.27" layer="96" rot="R90" display="off"/>
-</instance>
+<instance part="R22" gate="G$1" x="22.86" y="58.42" rot="R90">
+<attribute name="DIGIKEY" x="22.86" y="58.42" size="1.27" layer="96" rot="R90" display="off"/>
+</instance>
+<instance part="P+10" gate="VCC" x="22.86" y="78.74"/>
 </instances>
 <busses>
@@
 <wire x1="114.3" y1="167.64" x2="114.3" y2="170.18" width="0.1524" layer="91"/>
 </segment>
+<segment>
+<pinref part="D4" gate="G$1" pin="A"/>
+<pinref part="P+10" gate="VCC" pin="VCC"/>
+<wire x1="22.86" y1="73.66" x2="22.86" y2="76.2" width="0.1524" layer="91"/>
+</segment>
 </net>
 <net name="GND" class="0">
@@
 <pinref part="GND49" gate="1" pin="GND"/>
 <wire x1="48.26" y1="43.18" x2="48.26" y2="33.02" width="0.1524" layer="91"/>
-</segment>
-<segment>
-<pinref part="D4" gate="G$1" pin="C"/>
-<wire x1="22.86" y1="53.34" x2="22.86" y2="50.8" width="0.1524" layer="91"/>
-<pinref part="GND50" gate="1" pin="GND"/>
 </segment>
 <segment>
@@
 </segment>
 </net>
-<net name="N$63" class="0">
-<segment>
-<pinref part="D4" gate="G$1" pin="A"/>
-<wire x1="22.86" y1="60.96" x2="22.86" y2="63.5" width="0.1524" layer="91"/>
+<net name="N$64" class="0">
+<segment>
+<pinref part="U6" gate="G$1" pin="P13"/>
+<wire x1="33.02" y1="68.58" x2="50.8" y2="68.58" width="0.1524" layer="91"/>
+<wire x1="22.86" y1="50.8" x2="33.02" y2="50.8" width="0.1524" layer="91"/>
+<wire x1="33.02" y1="50.8" x2="33.02" y2="68.58" width="0.1524" layer="91"/>
 <pinref part="R22" gate="G$1" pin="1"/>
-</segment>
-</net>
-<net name="N$64" class="0">
-<segment>
-<wire x1="22.86" y1="73.66" x2="22.86" y2="78.74" width="0.1524" layer="91"/>
-<wire x1="22.86" y1="78.74" x2="35.56" y2="78.74" width="0.1524" layer="91"/>
-<wire x1="35.56" y1="78.74" x2="35.56" y2="68.58" width="0.1524" layer="91"/>
-<pinref part="U6" gate="G$1" pin="P13"/>
-<wire x1="35.56" y1="68.58" x2="50.8" y2="68.58" width="0.1524" layer="91"/>
-<pinref part="R22" gate="G$1" pin="2"/>
+<wire x1="22.86" y1="50.8" x2="22.86" y2="53.34" width="0.1524" layer="91"/>
 </segment>
 </net>
@@
 </segment>
 </net>
+<net name="N$63" class="0">
+<segment>
+<pinref part="D4" gate="G$1" pin="C"/>
+<pinref part="R22" gate="G$1" pin="2"/>
+<wire x1="22.86" y1="63.5" x2="22.86" y2="66.04" width="0.1524" layer="91"/>
+</segment>
+</net>

Commit message: updated schematic
Other:
- note added: "BeagleBone Black Header"
- note added: "CC2520. Index: 0, no amplifier"
- note added: "CC2520. Index: 1, with amplifier"
- note added: "Chip Select DeMux"
- note added: "EEPROM"
- note added: "LEDs"
- note added: "nRF51822"

Commit message: restore rev b
Parts:
- removed CS0, CS1, CS2: TEST_POINT_0.040IN, headers:TEST_POINT_0.040IN
- removed CS3, CS4: TPTP14SQ, testpad:TPTP14SQ
- removed J2: JUMPER-PTH-2-NO, SparkFun-Passives:JUMPER-PTH-2-NO
- removed SJ2: JUMPER-PAD-2-NC_BY_TRACE, SparkFun-Passives:JUMPER-PAD-2-NC_BY_TRACE
- added JP1: (no value), jumper:JP2Q
- added R18: 10k 1%, rcl:R-US_R0402
- added WRT: JUMPER-PTH-2-NO, SparkFun-Passives:JUMPER-PTH-2-NO
Connections:
- net CSE0 renamed SPIE0
- net CSE1 renamed SPIE1
- removed net !RESET2: P9/P8.UART4_RXD, U6.P04/AIN5
- removed net N$65: SJ2.1, U5.C
- removed net N$66: CS3.TP, U5.3
- removed net N$67: CS4.TP, U5.4
- removed net UARTRX: P9/P8.UART1_TXD, U6.P05/AIN6
- removed net UARTTX: P9/P8.UART1_RXD, U6.P06/AIN7/AREF1
- new net CS3: U5.3
- new net CS4: R18.1, U5.4
- new net CS5: U5.5
- new net CS6: U5.6
- new net CS7: U5.7
- new net P04: JP1.2, U6.P04/AIN5
- new net P05: JP1.4, U6.P05/AIN6
- new net P06: JP1.3, U6.P06/AIN7/AREF1
- net CS0: no longer CS0.TESTPOINT
- net CS1: no longer CS1.TESTPOINT
- net CS2: no longer CS2.TESTPOINT
- net GND: now also D4.C, U5.C, WRT.2; no longer J2.2, SJ2.2
- net N$31: now also WRT.1; no longer J2.1
- net N$63: now also D4.A, R22.1; no longer D4.C, R22.2
- net N$64: now also R22.2; no longer R22.1
- net P03: now also JP1.1
- net VCC: now also R18.2; no longer D4.A
Other:
- note removed: "BeagleBone Black Header"
- note removed: "CC2520. Index: 0, no amplifier"
- note removed: "CC2520. Index: 1, with amplifier"
- note removed: "Chip Select DeMux"
- note removed: "EEPROM"
- note removed: "LEDs"
- note removed: "nRF51822"
