File: hardware/eagle/bbb-cc2520/rev_c/bbb-cc2520.brd (EAGLE design)
At the start: 54.6 x 73.4 mm, 99 parts, among them J1 TC2030-IDC, J2 JUMPER-PTH-2-NO, P9/P8 BBB_HEADERS, U1 CC2520, U2 CC2520, U3 CAT24C256WI-GT3, U4 CC2591, U5 CD4051B-53B, U6 NRF51822QF, X1 NX2520SA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

Commit message: board cleaned up
Parts:
- removed R23: 12k, passives:0603-RES
- added R18: 56k 1%, rcl:R0402
- C1: value 1pF -> 0.8pF; device rcl:C0402 -> passives:0402_CAP
- C11, C12, C13: value 1nF -> 27pF
- C14, C15, C16: value 100nF -> 1nF
- C17, C18: value 100nF -> 1nF; device rcl:C0402 -> passives:0402_CAP
- C19: value 100nF -> 2.2nF; device rcl:C0402 -> passives:0402_CAP
- C2: value 2.7pF -> 1pF
- C20: value 100nF -> 47nF; device rcl:C0402 -> passives:0402_CAP
- C23, C24: value 1uF -> 100nF; device rcl:C0603 -> rcl:C0402
- C25: value 2.2uF -> 100nF
- C26: value 0.1uF -> 100nF; device passives:0402_CAP -> rcl:C0402
- C27: value 1nF -> 100nF; device passives:0402_CAP -> rcl:C0402
- C28: value 4.7uF -> 100nF; device passives:0402_CAP -> rcl:C0402
- C29: value 1uF -> 100nF; device passives:0402_CAP -> rcl:C0402
- C3: value 3pF -> 2.7pF
- C30: value 12pF -> 0.1uF
- C31: value 12pF -> 1uF
- C32: value 1nF -> 1uF; device passives:0402_CAP -> rcl:C0603
- C33: value 47nF -> 1uF; device passives:0402_CAP -> rcl:C0603
- C34: value 2.2nF -> 2.2uF; device passives:0402_CAP -> rcl:C0402
- C35: value 0.8pF -> 4.7uF
- C4: value 6.8pF -> 3pF
- C5: value 15pF -> 3.9pF
- C6: value 3.9pF -> 6.8pF
- C7, C8: value 27pF -> 12pF; device rcl:C0402 -> passives:0402_CAP
- C9: value 27pF -> 15pF
- L1, L2: value (none) -> 1nH; device SparkFun-Passives:0603 -> SparkFun-Passives:C0402
- L10: value 5.1nH -> 10uH; device SparkFun-Passives:C0402 -> passives:0603_CAP
- L12: device passives:0402_CAP -> SparkFun-Passives:0603
- L13: value 10uH -> (none); device passives:0603_CAP -> SparkFun-Passives:0603
- L5: value 1nH -> 1.1nH
- L6: value 1nH -> 1.5nH
- L7: value 1.1nH -> 2nH
- L8: value 1.5nH -> 5.1nH
- L9: value 2nH -> (none); device SparkFun-Passives:C0402 -> passives:0402_CAP
- R10: value 5.6k 5% -> 4.75k
- R12: value 10k 1% -> 5.6k 5%
- R13, R14: value 56k 1% -> 10k 1%
- R15: value 330k 1% -> 10k 1%
- R16: value 1M 1% -> 10k 1%
- R17: value 1M 1% -> 12k; device rcl:R0402 -> passives:0603-RES
- R19: value 10k 1% -> 56k 1%
- R20: value 10k 1% -> 330k 1%
- R21: value 10k 1% -> 1M 1%
- R22: value 470 -> 1M 1%
- R4: value 1k 1% -> 470
- R6: value 4.3k -> 1k 1%
- R7: value 4.75k -> 4.3k
- moved R13 55.4 mm to (7.87, 69.1), turned to 90 degrees
- moved C32 55.0 mm to (11.9, 11.4), turned to 180 degrees
- moved R7 54.7 mm to (45.5, 21.7)
- moved C8 54.6 mm to (31.8, 63.5), turned to 90 degrees
- moved C7 52.4 mm to (35.8, 63.5), turned to 270 degrees
- moved C25 47.5 mm to (10.9, 66.0)
- moved R4 47.2 mm to (46.7, 67.8), turned to 90 degrees
- moved C17 45.2 mm to (37.1, 61.5)
- moved C1 43.4 mm to (37.4, 59.1), turned to 90 degrees
- moved L10 42.4 mm to (27.2, 59.4), turned to 90 degrees
- moved L12 39.5 mm to (10.2, 22.6), turned to 180 degrees
- moved C11 36.6 mm to (8.13, 19.1), turned to 180 degrees
- moved C12 35.4 mm to (8.13, 14.2), turned to 180 degrees
- moved L9 35.3 mm to (25.7, 58.9), turned to 0 degrees
- moved C21 34.8 mm to (12.2, 13.3)
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- renumbered CS0 to TP0, CS1 to TP1, CS2 to TP2, CS3 to TP3, CS4 to TP4
Connections:
- net AVDD: now also C17.1, C31.1, L9.1; no longer C27.1, C29.1, L12.1
- net CS0: now also R14.1; no longer R19.1
- net CS1: now also R15.1; no longer R20.1
- net CS2: now also R16.1; no longer R21.1
- net DCC: now also L10.2; no longer L13.2
- net EN: now also R6.2; no longer R5.2
- net GND: now also C3.2, L1.1, L2.1, L4.2, R17.2, R18.1, R19.1, R21.1, R22.1, R7.1; no longer C5.2, L3.1, L4.1, L6.2, R13.1, R14.1, R16.1, R17.1, R23.2, R6.1
- net MISO: now also R21.2, R22.2; no longer R16.2, R17.2
- net N$11: now also C12.1; no longer C8.1
- net N$12: now also C24.1; no longer C17.1
- net N$13: now also C11.1; no longer C7.1
- net N$14: now also R18.2; no longer R13.2
- net N$29: now also R8.1; no longer R7.1
- net N$30: now also R9.1; no longer R8.1
- net N$31: now also R13.2; no longer R12.2
- net N$32: now also R10.1; no longer R9.1
- net N$38: now also C1.1; no longer C35.1
- net N$39: now also L10.1, L9.2; no longer L12.2, L13.1
- net N$40: now also C7.1; no longer C30.1
- net N$41: now also C8.1; no longer C31.1
- net N$42: now also C18.1; no longer C32.1
- net N$43: now also C20.1; no longer C33.1
- net N$44: now also L7.1; no longer L9.1
- net N$45: now also L3.1; no longer L5.1
- net N$46: now also C5.2, L2.2, L3.2; no longer C6.2, L4.2, L5.2
- net N$47: now also C4.2, L1.2, L7.2; no longer C3.2, L3.2, L9.2
- net N$48: now also L5.1, L8.1; no longer L10.1, L7.1
- net N$49: now also C14.1, C15.1, C16.1, C34.1, L8.2; no longer C11.1, C12.1, C13.1, C25.1, L10.2
- net N$5: now also C21.1, C22.1, C32.1, L12.1; no longer C14.1, C15.1, C16.1, L1.1
- net N$50: now also C9.1, L5.2; no longer C5.1, L7.2
- net N$51: now also L6.2; no longer L8.2
- net N$52: now also C3.1, C6.1, L4.1; no longer C2.1, C4.1, L6.1
- net N$53: now also C2.1, C6.2, L6.1; no longer C1.1, C4.2, L8.1
- net N$54: now also R7.2; no longer R6.2
- net N$55: now also R5.1; no longer R4.1
- net N$56: now also R6.1; no longer R5.1
- net N$57: now also C26.1, C27.1, C28.1, C33.1, L13.1; no longer C19.1, C20.1, C21.1, C24.1, L2.1
- net N$58: now also C29.1; no longer C22.1
- net N$60: now also C13.1; no longer C9.1
- net N$61: now also R19.2; no longer R14.2
- net N$62: now also R20.1; no longer R15.1
- net N$63: now also R4.2; no longer R22.2
- net N$64: now also R4.1; no longer R22.1
- net PAEN: now also R5.2; no longer R4.2
- net RF_N2: now also C5.1; no longer C6.1
- net RF_P2: now also C4.1; no longer C3.1
- net SCL: now also R11.1; no longer R10.1
- net SDA: now also R12.1; no longer R11.1
- net SWDCLK: now also R17.1; no longer R23.1
- net VCC: now also C25.1, C30.1, C35.1, L12.2, L13.2, R12.2, R13.1, R14.2, R16.2; no longer C18.1, C26.1, C28.1, L1.2, L2.2, R12.1, R19.2, R21.2, R7.2
- net VDD_PA: now also C19.1; no longer C34.1
Routing:
- net VCC: track 43.8 -> 44.9 mm
- net GND: track 21.7 -> 21.9 mm, vias 265 -> 267
