File: hardware/eagle/bbb-cc2520/rev_c/bbb-cc2520.sch (EAGLE design)
At the start: 98 parts, among them J1 TC2030-IDC, J2 JUMPER-PTH-2-NO, P9/P8 BBB_HEADERS, U1 CC2520, U2 CC2520, U3 CAT24C256WI-GT3, U4 CC2591, U5 CD4051B-53B, U6 NRF51822QF, X1 NX2520SA, X2 NX2520SA, X3 16MHz

Commit message: board cleaned up
Parts:
- removed R23: 12k, passives:RESISTOR
- added R18: 56k 1%, rcl:R-US_R0402
- C1: value 1pF -> 0.8pF; device rcl:C-EUC0402 -> passives:CAPACITOR; DIGIKEY 490-1318-1-ND -> 490-5419-1-ND
- C11, C12, C13: value 1nF -> 27pF; DIGIKEY 490-1318-1-ND -> 490-5869-1-ND
- C14, C15, C16: value 100nF -> 1nF
- C17, C18: value 100nF -> 1nF; device rcl:C-EUC0402 -> passives:CAPACITOR; DIGIKEY 490-1318-1-ND -> 490-1303-1-ND
- C19: value 100nF -> 2.2nF; device rcl:C-EUC0402 -> passives:CAPACITOR; DIGIKEY 490-1318-1-ND -> 490-5419-1-ND
- C2: value 2.7pF -> 1pF
- C20: value 100nF -> 47nF; device rcl:C-EUC0402 -> passives:CAPACITOR; DIGIKEY 490-1318-1-ND -> 445-1264-1-ND
- C23, C24: value 1uF -> 100nF; device rcl:C-EUC0603 -> rcl:C-EUC0402; DIGIKEY 490-1550-1-ND -> 490-1318-1-ND
- C25: value 2.2uF -> 100nF
- C26: value 0.1uF -> 100nF; device passives:CAPACITOR -> rcl:C-EUC0402; DIGIKEY 445-4952-1-ND -> 490-1318-1-ND
- C27: value 1nF -> 100nF; device passives:CAPACITOR -> rcl:C-EUC0402; DIGIKEY 490-1303-1-ND -> 490-1318-1-ND
- C28: value 4.7uF -> 100nF; device passives:CAPACITOR -> rcl:C-EUC0402; DIGIKEY 445-5947-1-ND -> 490-1318-1-ND
- C29: value 1uF -> 100nF; device passives:CAPACITOR -> rcl:C-EUC0402; DIGIKEY 1276-1513-1-ND -> 490-1318-1-ND
- C3: value 3pF -> 2.7pF
- C30: value 12pF -> 0.1uF; DIGIKEY 490-6197-1-ND -> 445-4952-1-ND
- C31: value 12pF -> 1uF; DIGIKEY 490-6197-1-ND -> 1276-1513-1-ND
- C32: value 1nF -> 1uF; device passives:CAPACITOR -> rcl:C-EUC0603; DIGIKEY 490-1303-1-ND -> 490-1550-1-ND
- C33: value 47nF -> 1uF; device passives:CAPACITOR -> rcl:C-EUC0603; DIGIKEY 445-1264-1-ND -> 490-1550-1-ND
- C34: value 2.2nF -> 2.2uF; device passives:CAPACITOR -> rcl:C-EUC0402; DIGIKEY 490-5419-1-ND -> 490-1318-1-ND
- C35: value 0.8pF -> 4.7uF; DIGIKEY 490-5419-1-ND -> 445-5947-1-ND
- C4: value 6.8pF -> 3pF
- C5: value 15pF -> 3.9pF
- C6: value 3.9pF -> 6.8pF
- C7, C8: value 27pF -> 12pF; device rcl:C-EUC0402 -> passives:CAPACITOR; DIGIKEY 490-5869-1-ND -> 490-6197-1-ND
- C9: value 27pF -> 15pF; DIGIKEY 490-5869-1-ND -> 490-1318-1-ND
- L1, L2: value (none) -> 1nH; device SparkFun-Passives:INDUCTOR0603 -> SparkFun-Passives:INDUCTOR0402; DIGIKEY 490-1015-1-ND -> (none)
- L10: value 5.1nH -> 10uH; device SparkFun-Passives:INDUCTOR0402 -> passives:INDUCTOR0603; DIGIKEY (none) -> 490-4025-1-ND
- L12: device passives:INDUCTOR0402 -> SparkFun-Passives:INDUCTOR0603; DIGIKEY 587-1521-1-ND -> 490-1015-1-ND
- L13: value 10uH -> (none); device passives:INDUCTOR0603 -> SparkFun-Passives:INDUCTOR0603; DIGIKEY 490-4025-1-ND -> 490-1015-1-ND
- L5: value 1nH -> 1.1nH
- L6: value 1nH -> 1.5nH
- L7: value 1.1nH -> 2nH
- L8: value 1.5nH -> 5.1nH
- L9: value 2nH -> (none); device SparkFun-Passives:INDUCTOR0402 -> passives:INDUCTOR0402; DIGIKEY (none) -> 587-1521-1-ND
- R10: value 5.6k 5% -> 4.75k
- R12: value 10k 1% -> 5.6k 5%
- R13, R14: value 56k 1% -> 10k 1%; DIGIKEY P56.0KLCT-ND -> RHM1.00MCDCT-ND
- R15: value 330k 1% -> 10k 1%; DIGIKEY P56.0KLCT-ND -> RHM1.00MCDCT-ND
- R16: value 1M 1% -> 10k 1%
- R17: value 1M 1% -> 12k; device rcl:R-US_R0402 -> passives:RESISTOR; DIGIKEY RHM1.00MCDCT-ND -> RHM12.0KCDCT-ND
- R19: value 10k 1% -> 56k 1%; DIGIKEY RHM1.00MCDCT-ND -> P56.0KLCT-ND
- R20: value 10k 1% -> 330k 1%; DIGIKEY RHM1.00MCDCT-ND -> P56.0KLCT-ND
- R21: value 10k 1% -> 1M 1%
- R22: value 470 -> 1M 1%; DIGIKEY RHM470JCT-ND -> RHM1.00MCDCT-ND
- R4: value 1k 1% -> 470; DIGIKEY P56.0KLCT-ND -> RHM470JCT-ND
- R6: value 4.3k -> 1k 1%
- R7: value 4.75k -> 4.3k; DIGIKEY RHM1.00MCDCT-ND -> P56.0KLCT-ND
- renumbered CS0 to TP0, CS1 to TP1, CS2 to TP2, CS3 to TP3, CS4 to TP4
Connections:
- net AVDD: now also C17.1, C31.1, L9.1; no longer C27.1, C29.1, L12.1
- net CS0: now also R14.1; no longer R19.1
- net CS1: now also R15.1; no longer R20.1
- net CS2: now also R16.1; no longer R21.1
- net DCC: now also L10.2; no longer L13.2
- net EN: now also R6.2; no longer R5.2
- net GND: now also C3.2, L1.1, L2.1, L4.2, R17.2, R18.1, R19.1, R21.1, R22.1, R7.1; no longer C5.2, L3.1, L4.1, L6.2, R13.1, R14.1, R16.1, R17.1, R23.2, R6.1
- net MISO: now also R21.2, R22.2; no longer R16.2, R17.2
- net N$11: now also C12.1; no longer C8.1
- net N$12: now also C24.1; no longer C17.1
- net N$13: now also C11.1; no longer C7.1
- net N$14: now also R18.2; no longer R13.2
- net N$29: now also R8.1; no longer R7.1
- net N$30: now also R9.1; no longer R8.1
- net N$31: now also R13.2; no longer R12.2
- net N$32: now also R10.1; no longer R9.1
- net N$38: now also C1.1; no longer C35.1
- net N$39: now also L10.1, L9.2; no longer L12.2, L13.1
- net N$40: now also C7.1; no longer C30.1
- net N$41: now also C8.1; no longer C31.1
- net N$42: now also C18.1; no longer C32.1
- net N$43: now also C20.1; no longer C33.1
- net N$44: now also L7.1; no longer L9.1
- net N$45: now also L3.1; no longer L5.1
- net N$46: now also C5.2, L2.2, L3.2; no longer C6.2, L4.2, L5.2
- net N$47: now also C4.2, L1.2, L7.2; no longer C3.2, L3.2, L9.2
- net N$48: now also L5.1, L8.1; no longer L10.1, L7.1
- net N$49: now also C14.1, C15.1, C16.1, C34.1, L8.2; no longer C11.1, C12.1, C13.1, C25.1, L10.2
- net N$5: now also C21.1, C22.1, C32.1, L12.1; no longer C14.1, C15.1, C16.1, L1.1
- net N$50: now also C9.1, L5.2; no longer C5.1, L7.2
- net N$51: now also L6.2; no longer L8.2
- net N$52: now also C3.1, C6.1, L4.1; no longer C2.1, C4.1, L6.1
- net N$53: now also C2.1, C6.2, L6.1; no longer C1.1, C4.2, L8.1
- net N$54: now also R7.2; no longer R6.2
- net N$55: now also R5.1; no longer R4.1
- net N$56: now also R6.1; no longer R5.1
- net N$57: now also C26.1, C27.1, C28.1, C33.1, L13.1; no longer C19.1, C20.1, C21.1, C24.1, L2.1
- net N$58: now also C29.1; no longer C22.1
- net N$60: now also C13.1; no longer C9.1
- net N$61: now also R19.2; no longer R14.2
- net N$62: now also R20.1; no longer R15.1
- net N$63: now also R4.2; no longer R22.2
- net N$64: now also R4.1; no longer R22.1
- net PAEN: now also R5.2; no longer R4.2
- net RF_N2: now also C5.1; no longer C6.1
- net RF_P2: now also C4.1; no longer C3.1
- net SCL: now also R11.1; no longer R10.1
- net SDA: now also R12.1; no longer R11.1
- net SWDCLK: now also R17.1; no longer R23.1
- net VCC: now also C25.1, C30.1, C35.1, L12.2, L13.2, R12.2, R13.1, R14.2, R16.2; no longer C18.1, C26.1, C28.1, L1.2, L2.2, R12.1, R19.2, R21.2, R7.2
- net VDD_PA: now also C19.1; no longer C34.1
