File: hardware/eagle/bbb-cc2520/rev_d/bbb-cc2520.sch (EAGLE design)
At the start: 97 parts, among them J1 TC2030-IDC, J2 JUMPER-PTH-2-NO, P9/P8 BBB_HEADERS, U1 CC2520, U2 CC2520, U3 CAT24C256WI-GT3, U4 CC2591, U5 CD4051B-53B, U6 NRF51822QF, X1 NX2520SA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

Commit message: committing changes to gap
Connections:
- removed net A0: U6.P26/AIN0/XL2
- removed net A1: U6.P27/AIN1/XL1
- removed net CC0_GPIO0: U1.GPIO0
- removed net CC0_GPIO5: U1.GPIO5
- removed net P03: U6.P03/AIN4
- removed net P12: U6.P12
- removed net P24: U6.P24
- removed net P25: U6.P25
- removed net PROG_RX: U6.P28
- removed net PROG_TX: U6.P29
Changed lines of the file:
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@@
-</segment>
-</net>
-<net name="CC0_GPIO5" class="0">
-<segment>
-<pinref part="U1" gate="G$1" pin="GPIO5"/>
-<wire x1="73.66" y1="99.06" x2="71.12" y2="99.06" width="0.1524" layer="91"/>
-<label x="71.12" y="99.06" size="1.27" layer="95" rot="R180" xref="yes"/>
-</segment>
-</net>
-<net name="CC0_GPIO0" class="0">
-<segment>
-<pinref part="U1" gate="G$1" pin="GPIO0"/>
-<wire x1="73.66" y1="86.36" x2="71.12" y2="86.36" width="0.1524" layer="91"/>
-<label x="71.12" y="86.36" size="1.27" layer="95" rot="R180" xref="yes"/>
 </segment>
 </net>
@@
 </segment>
 </net>
-<net name="P12" class="0">
-<segment>
-<pinref part="U6" gate="G$1" pin="P12"/>
-<wire x1="50.8" y1="71.12" x2="48.26" y2="71.12" width="0.1524" layer="91"/>
-<label x="48.26" y="71.12" size="1.27" layer="95" rot="R180" xref="yes"/>
-</segment>
-</net>
-<net name="PROG_RX" class="0">
-<segment>
-<pinref part="U6" gate="G$1" pin="P28"/>
-<wire x1="96.52" y1="76.2" x2="99.06" y2="76.2" width="0.1524" layer="91"/>
-<label x="99.06" y="76.2" size="1.27" layer="95" xref="yes"/>
-</segment>
-</net>
-<net name="PROG_TX" class="0">
-<segment>
-<pinref part="U6" gate="G$1" pin="P29"/>
-<wire x1="96.52" y1="73.66" x2="99.06" y2="73.66" width="0.1524" layer="91"/>
-<label x="99.06" y="73.66" size="1.27" layer="95" xref="yes"/>
-</segment>
-</net>
-<net name="P25" class="0">
-<segment>
-<pinref part="U6" gate="G$1" pin="P25"/>
-<wire x1="96.52" y1="83.82" x2="99.06" y2="83.82" width="0.1524" layer="91"/>
-<label x="99.06" y="83.82" size="1.27" layer="95" xref="yes"/>
-</segment>
-</net>
-<net name="P24" class="0">
-<segment>
-<pinref part="U6" gate="G$1" pin="P24"/>
-<wire x1="96.52" y1="86.36" x2="99.06" y2="86.36" width="0.1524" layer="91"/>
-<label x="99.06" y="86.36" size="1.27" layer="95" xref="yes"/>
-</segment>
-</net>
-<net name="A1" class="0">
-<segment>
-<pinref part="U6" gate="G$1" pin="P27/AIN1/XL1"/>
-<wire x1="96.52" y1="78.74" x2="99.06" y2="78.74" width="0.1524" layer="91"/>
-<label x="99.06" y="78.74" size="1.27" layer="95" xref="yes"/>
-</segment>
-</net>
-<net name="A0" class="0">
-<segment>
-<pinref part="U6" gate="G$1" pin="P26/AIN0/XL2"/>
-<wire x1="96.52" y1="81.28" x2="99.06" y2="81.28" width="0.1524" layer="91"/>
-<label x="99.06" y="81.28" size="1.27" layer="95" xref="yes"/>
-</segment>
-</net>
 <net name="UARTTX" class="0">
 <segment>
@@
 <wire x1="50.8" y1="93.98" x2="48.26" y2="93.98" width="0.1524" layer="91"/>
 <label x="48.26" y="93.98" size="1.27" layer="95" rot="R180" xref="yes"/>
-</segment>
-</net>
-<net name="P03" class="0">
-<segment>
-<pinref part="U6" gate="G$1" pin="P03/AIN4"/>
-<wire x1="50.8" y1="96.52" x2="48.26" y2="96.52" width="0.1524" layer="91"/>
-<label x="48.26" y="96.52" size="1.27" layer="95" rot="R180" xref="yes"/>
 </segment>
 </net>
@@
 <pinref part="P+7" gate="1" pin="VCC"/>
 <wire x1="165.1" y1="137.16" x2="165.1" y2="120.65" width="0.1524" layer="91"/>
-</segment>
-<segment>
-<pinref part="R15" gate="G$1" pin="2"/>
-<wire x1="200.66" y1="129.54" x2="200.66" y2="132.08" width="0.1524" layer="91"/>
-<pinref part="R16" gate="G$1" pin="2"/>
-<wire x1="200.66" y1="132.08" x2="208.28" y2="132.08" width="0.1524" layer="91"/>
-<wire x1="208.28" y1="132.08" x2="208.28" y2="129.54" width="0.1524" layer="91"/>
-<wire x1="200.66" y1="132.08" x2="193.04" y2="132.08" width="0.1524" layer="91"/>
-<pinref part="P+8" gate="1" pin="VCC"/>
-<wire x1="193.04" y1="132.08" x2="193.04" y2="137.16" width="0.1524" layer="91"/>
-<pinref part="R14" gate="G$1" pin="2"/>
-<wire x1="193.04" y1="137.16" x2="193.04" y2="129.54" width="0.1524" layer="91"/>
 </segment>
 <segment>
@@
 <wire x1="78.74" y1="63.5" x2="78.74" y2="60.96" width="0.1524" layer="91"/>
 </segment>
+<segment>
+<pinref part="R15" gate="G$1" pin="2"/>
+<wire x1="200.66" y1="129.54" x2="200.66" y2="132.08" width="0.1524" layer="91"/>
+<pinref part="R16" gate="G$1" pin="2"/>
+<wire x1="200.66" y1="132.08" x2="208.28" y2="132.08" width="0.1524" layer="91"/>
+<wire x1="208.28" y1="132.08" x2="208.28" y2="129.54" width="0.1524" layer="91"/>
+<wire x1="200.66" y1="132.08" x2="193.04" y2="132.08" width="0.1524" layer="91"/>
+<pinref part="R14" gate="G$1" pin="2"/>
+<junction x="200.66" y="132.08"/>
+<wire x1="193.04" y1="132.08" x2="193.04" y2="129.54" width="0.1524" layer="91"/>
+<pinref part="P+8" gate="1" pin="VCC"/>
+<wire x1="193.04" y1="137.16" x2="193.04" y2="132.08" width="0.1524" layer="91"/>
+<junction x="193.04" y="132.08"/>
+</segment>
 </net>
 <net name="SPI0_CS0_0" class="0">
@@
 </sheet>
 </sheets>
+<errors>
+</errors>
 </schematic>
 </drawing>
